File: Platform/PowerManagement.sch (KiCad schematic (older format))
At the start: 17 parts

Commit message: Added RTC and EEPROM
Parts:
- gave numbers to parts that had none: 17
Changed lines of the file:
@@
 $EndDescr
 $Comp
-L power:+12V #PWR?
+L power:+12V #PWR0101
 U 1 1 5FA6C6C2
 P 5150 1750
-F 0 "#PWR?" H 5150 1600 50  0001 C CNN
+F 0 "#PWR0101" H 5150 1600 50  0001 C CNN
 F 1 "+12V" H 5165 1923 50  0000 C CNN
 F 2 "" H 5150 1750 50  0001 C CNN
@@
 $EndComp
 $Comp
-L power:GND #PWR?
+L power:GND #PWR0102
 U 1 1 5FA6C9F6
 P 5150 2150
-F 0 "#PWR?" H 5150 1900 50  0001 C CNN
+F 0 "#PWR0102" H 5150 1900 50  0001 C CNN
 F 1 "GND" H 5155 1977 50  0000 C CNN
 F 2 "" H 5150 2150 50  0001 C CNN
@@
 	5150 2000 5450 2000
 $Comp
-L power:PWR_FLAG #FLG?
+L power:PWR_FLAG #FLG0101
 U 1 1 5FA71D78
 P 5400 1400
-F 0 "#FLG?" H 5400 1475 50  0001 C CNN
+F 0 "#FLG0101" H 5400 1475 50  0001 C CNN
 F 1 "PWR_FLAG" H 5400 1573 50  0000 C CNN
 F 2 "" H 5400 1400 50  0001 C CNN
@@
 	5400 1400 5400 1900
 $Comp
-L power:PWR_FLAG #FLG?
+L power:PWR_FLAG #FLG0102
 U 1 1 5FA724DF
 P 5450 2550
-F 0 "#FLG?" H 5450 2625 50  0001 C CNN
+F 0 "#FLG0102" H 5450 2625 50  0001 C CNN
 F 1 "PWR_FLAG" H 5450 2723 50  0000 C CNN
 F 2 "" H 5450 2550 50  0001 C CNN
@@
 	5450 2550 5450 2000
 $Comp
-L Regulator_Linear:LM7805_TO220 U?
+L Regulator_Linear:LM7805_TO220 U1
 U 1 1 5FA72B80
 P 3100 4800
-F 0 "U?" H 3100 5042 50  0000 C CNN
+F 0 "U1" H 3100 5042 50  0000 C CNN
 F 1 "LM7805_TO220" H 3100 4951 50  0000 C CNN
 F 2 "Package_TO_SOT_THT:TO-220-3_Vertical" H 3100 5025 50  0001 C CIN
@@
 $EndComp
 $Comp
-L power:+12V #PWR?
+L power:+12V #PWR0103
 U 1 1 5FA73447
 P 2350 4550
-F 0 "#PWR?" H 2350 4400 50  0001 C CNN
+F 0 "#PWR0103" H 2350 4400 50  0001 C CNN
 F 1 "+12V" H 2365 4723 50  0000 C CNN
 F 2 "" H 2350 4550 50  0001 C CNN
@@
 	2350 4800 2500 4800
 $Comp
-L power:+5V #PWR?
+L power:+5V #PWR0104
 U 1 1 5FA73B37
 P 3800 4550
-F 0 "#PWR?" H 3800 4400 50  0001 C CNN
+F 0 "#PWR0104" H 3800 4400 50  0001 C CNN
 F 1 "+5V" H 3815 4723 50  0000 C CNN
 F 2 "" H 3800 4550 50  0001 C CNN
@@
 	3800 4800 3600 4800
 $Comp
-L power:GND #PWR?
+L power:GND #PWR0105
 U 1 1 5FA74A2F
 P 3100 5250
-F 0 "#PWR?" H 3100 5000 50  0001 C CNN
+F 0 "#PWR0105" H 3100 5000 50  0001 C CNN
 F 1 "GND" H 3105 5077 50  0000 C CNN
 F 2 "" H 3100 5250 50  0001 C CNN
@@
 	3100 5250 3100 5100
 $Comp
-L Device:CP C?
+L Device:CP C1
 U 1 1 5FA7541C
 P 2500 5100
-F 0 "C?" H 2618 5146 50  0000 L CNN
+F 0 "C1" H 2618 5146 50  0000 L CNN
 F 1 "0.33uF" H 2618 5055 50  0000 L CNN
 F 2 "" H 2538 4950 50  0001 C CNN
@@
 Connection ~ 3100 5250
 $Comp
-L Device:CP C?
+L Device:CP C2
 U 1 1 5FA75BDB
 P 3600 4950
-F 0 "C?" H 3718 4996 50  0000 L CNN
+F 0 "C2" H 3718 4996 50  0000 L CNN
 F 1 "0.1uF" H 3718 4905 50  0000 L CNN
 F 2 "" H 3638 4800 50  0001 C CNN
@@
 Connection ~ 3100 5100
 $Comp
-L Regulator_Linear:LM317_TO-220 U?
+L Regulator_Linear:LM317_TO-220 U2
 U 1 1 5FA76F90
 P 7350 4300
-F 0 "U?" H 7350 4542 50  0000 C CNN
+F 0 "U2" H 7350 4542 50  0000 C CNN
 F 1 "LM317_TO-220" H 7350 4451 50  0000 C CNN
 F 2 "Package_TO_SOT_THT:TO-220-3_Vertical" H 7350 4550 50  0001 C CIN
@@
 $EndComp
 $Comp
-L power:+12V #PWR?
+L power:+12V #PWR0106
 U 1 1 5FA77820
 P 6050 3850
-F 0 "#PWR?" H 6050 3700 50  0001 C CNN
+F 0 "#PWR0106" H 6050 3700 50  0001 C CNN
 F 1 "+12V" H 6065 4023 50  0000 C CNN
 F 2 "" H 6050 3850 50  0001 C CNN
@@
 	6050 4300 6550 4300
 $Comp
-L power:+3.3V #PWR?
+L power:+3.3V #PWR0107
 U 1 1 5FA788F5
 P 9250 4350
-F 0 "#PWR?" H 9250 4200 50  0001 C CNN
+F 0 "#PWR0107" H 9250 4200 50  0001 C CNN
 F 1 "+3.3V" V 9265 4478 50  0000 L CNN
 F 2 "" H 9250 4350 50  0001 C CNN
@@
 	9250 4300 9250 4350
 $Comp
-L Device:CP C?
+L Device:CP C3
 U 1 1 5FA79CE3
 P 6550 4900
-F 0 "C?" H 6668 4946 50  0000 L CNN
+F 0 "C3" H 6668 4946 50  0000 L CNN
 F 1 "0.1uF" H 6668 4855 50  0000 L CNN
 F 2 "" H 6588 4750 50  0001 C CNN
@@
 $EndComp
 $Comp
-L Device:CP C?
+L Device:CP C5
 U 1 1 5FA7A319
 P 9250 5050
-F 0 "C?" H 9368 5096 50  0000 L CNN
+F 0 "C5" H 9368 5096 50  0000 L CNN
 F 1 "1uF" H 9368 5005 50  0000 L CNN
 F 2 "" H 9288 4900 50  0001 C CNN
@@
 $EndComp
 $Comp
-L Device:CP C?
+L Device:CP C4
 U 1 1 5FA7BC81
 P 8200 5300
-F 0 "C?" H 8318 5346 50  0000 L CNN
+F 0 "C4" H 8318 5346 50  0000 L CNN
 F 1 "10uF" H 8318 5255 50  0000 L CNN
 F 2 "" H 8238 5150 50  0001 C CNN
@@
 $EndComp
 $Comp
-L Diode:1N4001 D?
+L Diode:1N4001 D1
 U 1 1 5FA7C443
 P 8200 4700
-F 0 "D?" V 8154 4780 50  0000 L CNN
+F 0 "D1" V 8154 4780 50  0000 L CNN
 F 1 "1N4001" V 8245 4780 50  0000 L CNN
 F 2 "Diode_THT:D_DO-41_SOD81_P10.16mm_Horizontal" H 8200 4525 50  0001 C CNN
@@
 	8200 5450 8200 5550
 $Comp
-L power:GND #PWR?
+L power:GND #PWR0108
 U 1 1 5FA84744
 P 7350 5550
-F 0 "#PWR?" H 7350 5300 50  0001 C CNN
+F 0 "#PWR0108" H 7350 5300 50  0001 C CNN
 F 1 "GND" H 7355 5377 50  0000 C CNN
 F 2 "" H 7350 5550 50  0001 C CNN
@@
 Connection ~ 8200 5550
 $Comp
-L Device:R R?
+L Device:R R1
 U 1 1 5FA8798A
 P 7850 4650
-F 0 "R?" H 7920 4696 50  0000 L CNN
+F 0 "R1" H 7920 4696 50  0000 L CNN
 F 1 "1K" H 7920 4605 50  0000 L CNN
 F 2 "" V 7780 4650 50  0001 C CNN
@@
 $EndComp
 $Comp
-L Device:R R?
+L Device:R R2
 U 1 1 5FA87CE9
 P 7850 5250
-F 0 "R?" H 7920 5296 50  0000 L CNN
+F 0 "R2" H 7920 5296 50  0000 L CNN
 F 1 "5.1K" H 7920 5205 50  0000 L CNN
 F 2 "" V 7780 5250 50  0001 C CNN
@@
 12V to 3v3 LDO regulation
 $Comp
-L Connector_Generic:Conn_01x02 J?
+L Connector_Generic:Conn_01x02 J1
 U 1 1 5FAB8A00
 P 4650 2000
-F 0 "J?" H 4568 1675 50  0000 C CNN
+F 0 "J1" H 4568 1675 50  0000 C CNN
 F 1 "12V INPUT" H 4568 1766 50  0000 C CNN
 F 2 "" H 4650 2000 50  0001 C CNN
@@
 Connection ~ 5150 2000
 $Comp
-L Connector:Screw_Terminal_01x02 J?
+L Connector:Screw_Terminal_01x02 J2
 U 1 1 5FABBF92
 P 6200 1900
-F 0 "J?" H 6280 1892 50  0000 L CNN
+F 0 "J2" H 6280 1892 50  0000 L CNN
 F 1 "12V_INPUT" H 6280 1801 50  0000 L CNN
 F 2 "" H 6200 1900 50  0001 C CNN
@@
 Connection ~ 5450 2000
 $Comp
-L Mechanical:MountingHole H?
+L Mechanical:MountingHole H1
 U 1 1 5FABED39
 P 8150 1450
-F 0 "H?" H 8250 1496 50  0000 L CNN
+F 0 "H1" H 8250 1496 50  0000 L CNN
 F 1 "MountingHole" H 8250 1405 50  0000 L CNN
 F 2 "" H 8150 1450 50  0001 C CNN
@@
 $EndComp
 $Comp
-L Mechanical:MountingHole H?
+L Mechanical:MountingHole H2
 U 1 1 5FABF30F
 P 8850 1450
-F 0 "H?" H 8950 1496 50  0000 L CNN
+F 0 "H2" H 8950 1496 50  0000 L CNN
 F 1 "MountingHole" H 8950 1405 50  0000 L CNN
 F 2 "" H 8850 1450 50  0001 C CNN
@@
 $EndComp
 $Comp
-L Mechanical:MountingHole H?
+L Mechanical:MountingHole H3
 U 1 1 5FABF685
 P 9550 1450
-F 0 "H?" H 9650 1496 50  0000 L CNN
+F 0 "H3" H 9650 1496 50  0000 L CNN
 F 1 "MountingHole" H 9650 1405 50  0000 L CNN
 F 2 "" H 9550 1450 50  0001 C CNN
@@
 $EndComp
 $Comp
-L Mechanical:MountingHole H?
+L Mechanical:MountingHole H4
 U 1 1 5FABF99D
 P 10250 1450
-F 0 "H?" H 10350 1496 50  0000 L CNN
+F 0 "H4" H 10350 1496 50  0000 L CNN
 F 1 "MountingHole" H 10350 1405 50  0000 L CNN
 F 2 "" H 10250 1450 50  0001 C CNN
@@
 $EndComp
 $Comp
-L power:GND #PWR?
+L power:GND #PWR0109
 U 1 1 5FABFC8F
 P 8150 1500
-F 0 "#PWR?" H 8150 1250 50  0001 C CNN
+F 0 "#PWR0109" H 8150 1250 50  0001 C CNN
 F 1 "GND" H 8155 1327 50  0000 C CNN
 F 2 "" H 8150 1500 50  0001 C CNN
@@
 $EndComp
 $Comp
-L power:GND #PWR?
+L power:GND #PWR0110
 U 1 1 5FAC713B
 P 8850 1500
-F 0 "#PWR?" H 8850 1250 50  0001 C CNN
+F 0 "#PWR0110" H 8850 1250 50  0001 C CNN
 F 1 "GND" H 8855 1327 50  0000 C CNN
 F 2 "" H 8850 1500 50  0001 C CNN
@@
 $EndComp
 $Comp
-L power:GND #PWR?
+L power:GND #PWR0111
 U 1 1 5FAC7558
 P 9550 1500
-F 0 "#PWR?" H 9550 1250 50  0001 C CNN
+F 0 "#PWR0111" H 9550 1250 50  0001 C CNN
 F 1 "GND" H 9555 1327 50  0000 C CNN
 F 2 "" H 9550 1500 50  0001 C CNN
@@
 $EndComp
 $Comp
-L power:GND #PWR?
+L power:GND #PWR0112
 U 1 1 5FAC79A8
 P 10250 1500
-F 0 "#PWR?" H 10250 1250 50  0001 C CNN
+F 0 "#PWR0112" H 10250 1250 50  0001 C CNN
 F 1 "GND" H 10255 1327 50  0000 C CNN
 F 2 "" H 10250 1500 50  0001 C CNN
@@
 	11050 1050 7900 1050
 $Comp
-L Connector:Barrel_Jack J?
+L Connector:Barrel_Jack J3
 U 1 1 5FACD235
 P 6350 1450
-F 0 "J?" H 6120 1408 50  0000 R CNN
+F 0 "J3" H 6120 1408 50  0000 R CNN
 F 1 "Barrel_Jack" H 6120 1499 50  0000 R CNN
 F 2 "" H 6400 1410 50  0001 C CNN

Commit message: changes
Connections:
- wire segments 58 -> 59
Changed lines of the file:
@@
 $EndDescr
 $Comp
-L power:+12V #PWR0101
+L power:+12V #PWR04
 U 1 1 5FA6C6C2
 P 5150 1750
-F 0 "#PWR0101" H 5150 1600 50  0001 C CNN
+F 0 "#PWR04" H 5150 1600 50  0001 C CNN
 F 1 "+12V" H 5165 1923 50  0000 C CNN
 F 2 "" H 5150 1750 50  0001 C CNN
@@
 $EndComp
 $Comp
-L power:GND #PWR0102
+L power:GND #PWR05
 U 1 1 5FA6C9F6
 P 5150 2150
-F 0 "#PWR0102" H 5150 1900 50  0001 C CNN
+F 0 "#PWR05" H 5150 1900 50  0001 C CNN
 F 1 "GND" H 5155 1977 50  0000 C CNN
 F 2 "" H 5150 2150 50  0001 C CNN
@@
 	5150 2000 5450 2000
 $Comp
-L power:PWR_FLAG #FLG0101
+L power:PWR_FLAG #FLG01
 U 1 1 5FA71D78
 P 5400 1400
-F 0 "#FLG0101" H 5400 1475 50  0001 C CNN
+F 0 "#FLG01" H 5400 1475 50  0001 C CNN
 F 1 "PWR_FLAG" H 5400 1573 50  0000 C CNN
 F 2 "" H 5400 1400 50  0001 C CNN
@@
 	5400 1400 5400 1900
 $Comp
-L power:PWR_FLAG #FLG0102
+L power:PWR_FLAG #FLG02
 U 1 1 5FA724DF
 P 5450 2550
-F 0 "#FLG0102" H 5450 2625 50  0001 C CNN
+F 0 "#FLG02" H 5450 2625 50  0001 C CNN
 F 1 "PWR_FLAG" H 5450 2723 50  0000 C CNN
 F 2 "" H 5450 2550 50  0001 C CNN
@@
 $EndComp
 $Comp
-L power:+12V #PWR0103
+L power:+12V #PWR01
 U 1 1 5FA73447
 P 2350 4550
-F 0 "#PWR0103" H 2350 4400 50  0001 C CNN
+F 0 "#PWR01" H 2350 4400 50  0001 C CNN
 F 1 "+12V" H 2365 4723 50  0000 C CNN
 F 2 "" H 2350 4550 50  0001 C CNN
@@
 	2350 4800 2500 4800
 $Comp
-L power:+5V #PWR0104
+L power:+5V #PWR03
 U 1 1 5FA73B37
 P 3800 4550
-F 0 "#PWR0104" H 3800 4400 50  0001 C CNN
+F 0 "#PWR03" H 3800 4400 50  0001 C CNN
 F 1 "+5V" H 3815 4723 50  0000 C CNN
 F 2 "" H 3800 4550 50  0001 C CNN
@@
 	3800 4800 3600 4800
 $Comp
-L power:GND #PWR0105
+L power:GND #PWR02
 U 1 1 5FA74A2F
 P 3100 5250
-F 0 "#PWR0105" H 3100 5000 50  0001 C CNN
+F 0 "#PWR02" H 3100 5000 50  0001 C CNN
 F 1 "GND" H 3105 5077 50  0000 C CNN
 F 2 "" H 3100 5250 50  0001 C CNN
@@
 $EndComp
 $Comp
-L power:+12V #PWR0106
+L power:+12V #PWR06
 U 1 1 5FA77820
 P 6050 3850
-F 0 "#PWR0106" H 6050 3700 50  0001 C CNN
+F 0 "#PWR06" H 6050 3700 50  0001 C CNN
 F 1 "+12V" H 6065 4023 50  0000 C CNN
 F 2 "" H 6050 3850 50  0001 C CNN
@@
 	6050 4300 6550 4300
 $Comp
-L power:+3.3V #PWR0107
+L power:+3.3V #PWR010
 U 1 1 5FA788F5
 P 9250 4350
-F 0 "#PWR0107" H 9250 4200 50  0001 C CNN
+F 0 "#PWR010" H 9250 4200 50  0001 C CNN
 F 1 "+3.3V" V 9265 4478 50  0000 L CNN
 F 2 "" H 9250 4350 50  0001 C CNN
@@
 	8200 5450 8200 5550
 $Comp
-L power:GND #PWR0108
+L power:GND #PWR07
 U 1 1 5FA84744
 P 7350 5550
-F 0 "#PWR0108" H 7350 5300 50  0001 C CNN
+F 0 "#PWR07" H 7350 5300 50  0001 C CNN
 F 1 "GND" H 7355 5377 50  0000 C CNN
 F 2 "" H 7350 5550 50  0001 C CNN
@@
 	1    0    0    -1
 $EndComp
-Wire Wire Line
-	7350 4600 7350 5550
 Wire Wire Line
 	8200 5550 7850 5550
@@
 $EndComp
 $Comp
-L power:GND #PWR0109
+L power:GND #PWR08
 U 1 1 5FABFC8F
 P 8150 1500
-F 0 "#PWR0109" H 8150 1250 50  0001 C CNN
+F 0 "#PWR08" H 8150 1250 50  0001 C CNN
 F 1 "GND" H 8155 1327 50  0000 C CNN
 F 2 "" H 8150 1500 50  0001 C CNN
@@
 $EndComp
 $Comp
-L power:GND #PWR0110
+L power:GND #PWR09
 U 1 1 5FAC713B
 P 8850 1500
-F 0 "#PWR0110" H 8850 1250 50  0001 C CNN
+F 0 "#PWR09" H 8850 1250 50  0001 C CNN
 F 1 "GND" H 8855 1327 50  0000 C CNN
 F 2 "" H 8850 1500 50  0001 C CNN
@@
 $EndComp
 $Comp
-L power:GND #PWR0111
+L power:GND #PWR011
 U 1 1 5FAC7558
 P 9550 1500
-F 0 "#PWR0111" H 9550 1250 50  0001 C CNN
+F 0 "#PWR011" H 9550 1250 50  0001 C CNN
 F 1 "GND" H 9555 1327 50  0000 C CNN
 F 2 "" H 9550 1500 50  0001 C CNN
@@
 $EndComp
 $Comp
-L power:GND #PWR0112
+L power:GND #PWR012
 U 1 1 5FAC79A8
 P 10250 1500
-F 0 "#PWR0112" H 10250 1250 50  0001 C CNN
+F 0 "#PWR012" H 10250 1250 50  0001 C CNN
 F 1 "GND" H 10255 1327 50  0000 C CNN
 F 2 "" H 10250 1500 50  0001 C CNN
@@
 Wire Wire Line
 	5150 2100 5150 2000
+Wire Wire Line
+	7350 4600 7350 4950
+Wire Wire Line
+	7350 4950 7850 4950
 $EndSCHEMATC

Commit message: Fixed ERC errors.
Parts:
- U2: symbol Regulator_Linear:LM317_TO-220 -> Platform-rescue:LM317_TO-220-Regulator_Linear
Connections:
- wire segments 59 -> 57
Changed lines of the file:
@@
 Wire Wire Line
 	5150 2150 5150 2100
-Wire Wire Line
-	5150 2000 5450 2000
 $Comp
 L power:PWR_FLAG #FLG01
@@
 	5400 1400 5400 1900
 $Comp
-L power:PWR_FLAG #FLG02
-U 1 1 5FA724DF
-P 5450 2550
-F 0 "#FLG02" H 5450 2625 50  0001 C CNN
-F 1 "PWR_FLAG" H 5450 2723 50  0000 C CNN
-F 2 "" H 5450 2550 50  0001 C CNN
-F 3 "~" H 5450 2550 50  0001 C CNN
-	1    5450 2550
-	-1   0    0    1
-$EndComp
-Wire Wire Line
-	5450 2550 5450 2000
-$Comp
 L Regulator_Linear:LM7805_TO220 U1
 U 1 1 5FA72B80
@@
 Connection ~ 3100 5100
 $Comp
-L Regulator_Linear:LM317_TO-220 U2
+L Platform-rescue:LM317_TO-220-Regulator_Linear U2
 U 1 1 5FA76F90
 P 7350 4300
@@
 	6000 1900 5750 1900
 Connection ~ 5400 1900
-Wire Wire Line
-	6000 2000 5450 2000
-Connection ~ 5450 2000
 $Comp
 L Mechanical:MountingHole H1
@@
 Wire Wire Line
 	7350 4950 7850 4950
+Wire Wire Line
+	5150 2000 6000 2000
 $EndSCHEMATC

Commit message: updated.
Parts:
- U2: symbol Platform-rescue:LM317_TO-220-Regulator_Linear -> Platform-rescue:LM317_TO-220-Regulator_Linear-Platform-rescue
Changed lines of the file:
@@
 Connection ~ 3100 5100
 $Comp
-L Platform-rescue:LM317_TO-220-Regulator_Linear U2
+L Platform-rescue:LM317_TO-220-Regulator_Linear-Platform-rescue U2
 U 1 1 5FA76F90
 P 7350 4300
