File: Platform/PowerManagement.sch (KiCad schematic (older format))
At the start: 29 parts, among them J1 12V INPUT, J2 12V_INPUT, J3 Barrel_Jack, J5 AC INPUT, J8 Conn_01x06, U1 LM7805_TO220, U2 LM317_TO-220, U4 NSL-32

Commit message: updated.
Parts:
- J8: footprint (none) -> Connector_PinHeader_2.54mm:PinHeader_1x06_P2.54mm_Vertical
Changed lines of the file:
@@
 F 0 "J8" H 2730 3592 50  0000 L CNN
 F 1 "Conn_01x06" H 2730 3501 50  0000 L CNN
-F 2 "" H 2650 3600 50  0001 C CNN
+F 2 "Connector_PinHeader_2.54mm:PinHeader_1x06_P2.54mm_Vertical" H 2650 3600 50  0001 C CNN
 F 3 "~" H 2650 3600 50  0001 C CNN
 	1    2650 3600

Commit message: GRM155R61C105KE01D
Parts:
- C1: value 0.33uF -> 0.33uF 330NF-0402; footprint (none) -> Capacitor_SMD:C_0402_1005Metric
- C2, C3: footprint (none) -> Capacitor_SMD:C_0402_1005Metric
- C4, C5: footprint (none) -> Capacitor_THT:CP_Radial_Tantal_D5.0mm_P5.00mm
- H1, H2, H3, H4: footprint (none) -> MountingHole:MountingHole_4mm
- J1, J2: footprint (none) -> Connector_PinHeader_2.54mm:PinHeader_1x02_P2.54mm_Vertical
- U2: symbol Platform-rescue:LM317_TO-220-Regulator_Linear-Platform-rescue -> Platform-rescue:LM317_TO-220-Regulator_Linear-Platform-rescue-Platform-rescue
Changed lines of the file:
@@
 P 2150 2250
 F 0 "C1" H 2268 2296 50  0000 L CNN
-F 1 "0.33uF" H 2268 2205 50  0000 L CNN
-F 2 "" H 2188 2100 50  0001 C CNN
+F 1 "0.33uF 330NF-0402" H 2268 2205 50  0000 L CNN
+F 2 "Capacitor_SMD:C_0402_1005Metric" H 2188 2100 50  0001 C CNN
 F 3 "~" H 2150 2250 50  0001 C CNN
 	1    2150 2250
@@
 F 0 "C2" H 3368 2146 50  0000 L CNN
 F 1 "0.1uF" H 3368 2055 50  0000 L CNN
-F 2 "" H 3288 1950 50  0001 C CNN
+F 2 "Capacitor_SMD:C_0402_1005Metric" H 3288 1950 50  0001 C CNN
 F 3 "~" H 3250 2100 50  0001 C CNN
 	1    3250 2100
@@
 Connection ~ 2750 2250
 $Comp
-L Platform-rescue:LM317_TO-220-Regulator_Linear-Platform-rescue U2
+L Platform-rescue:LM317_TO-220-Regulator_Linear-Platform-rescue-Platform-rescue U2
 U 1 1 5FA76F90
 P 7350 4300
@@
 F 0 "C3" H 6668 4946 50  0000 L CNN
 F 1 "0.1uF" H 6668 4855 50  0000 L CNN
-F 2 "" H 6588 4750 50  0001 C CNN
+F 2 "Capacitor_SMD:C_0402_1005Metric" H 6588 4750 50  0001 C CNN
 F 3 "~" H 6550 4900 50  0001 C CNN
 	1    6550 4900
@@
 F 0 "C5" H 9368 5096 50  0000 L CNN
 F 1 "1uF" H 9368 5005 50  0000 L CNN
-F 2 "" H 9288 4900 50  0001 C CNN
+F 2 "Capacitor_THT:CP_Radial_Tantal_D5.0mm_P5.00mm" H 9288 4900 50  0001 C CNN
 F 3 "~" H 9250 5050 50  0001 C CNN
 	1    9250 5050
@@
 F 0 "C4" H 8318 5346 50  0000 L CNN
 F 1 "10uF" H 8318 5255 50  0000 L CNN
-F 2 "" H 8238 5150 50  0001 C CNN
+F 2 "Capacitor_THT:CP_Radial_Tantal_D5.0mm_P5.00mm" H 8238 5150 50  0001 C CNN
 F 3 "~" H 8200 5300 50  0001 C CNN
 	1    8200 5300
@@
 F 0 "J1" H 4568 1675 50  0000 C CNN
 F 1 "12V INPUT" H 4568 1766 50  0000 C CNN
-F 2 "" H 4650 2000 50  0001 C CNN
+F 2 "Connector_PinHeader_2.54mm:PinHeader_1x02_P2.54mm_Vertical" H 4650 2000 50  0001 C CNN
 F 3 "~" H 4650 2000 50  0001 C CNN
 	1    4650 2000
@@
 F 0 "J2" H 6280 1892 50  0000 L CNN
 F 1 "12V_INPUT" H 6280 1801 50  0000 L CNN
-F 2 "" H 6200 1900 50  0001 C CNN
+F 2 "Connector_PinHeader_2.54mm:PinHeader_1x02_P2.54mm_Vertical" H 6200 1900 50  0001 C CNN
 F 3 "~" H 6200 1900 50  0001 C CNN
 	1    6200 1900
@@
 F 0 "H1" H 8250 1496 50  0000 L CNN
 F 1 "MountingHole" H 8250 1405 50  0000 L CNN
-F 2 "" H 8150 1450 50  0001 C CNN
+F 2 "MountingHole:MountingHole_4mm" H 8150 1450 50  0001 C CNN
 F 3 "~" H 8150 1450 50  0001 C CNN
 	1    8150 1450
@@
 F 0 "H2" H 8950 1496 50  0000 L CNN
 F 1 "MountingHole" H 8950 1405 50  0000 L CNN
-F 2 "" H 8850 1450 50  0001 C CNN
+F 2 "MountingHole:MountingHole_4mm" H 8850 1450 50  0001 C CNN
 F 3 "~" H 8850 1450 50  0001 C CNN
 	1    8850 1450
@@
 F 0 "H3" H 9650 1496 50  0000 L CNN
 F 1 "MountingHole" H 9650 1405 50  0000 L CNN
-F 2 "" H 9550 1450 50  0001 C CNN
+F 2 "MountingHole:MountingHole_4mm" H 9550 1450 50  0001 C CNN
 F 3 "~" H 9550 1450 50  0001 C CNN
 	1    9550 1450
@@
 F 0 "H4" H 10350 1496 50  0000 L CNN
 F 1 "MountingHole" H 10350 1405 50  0000 L CNN
-F 2 "" H 10250 1450 50  0001 C CNN
+F 2 "MountingHole:MountingHole_4mm" H 10250 1450 50  0001 C CNN
 F 3 "~" H 10250 1450 50  0001 C CNN
 	1    10250 1450

Commit message: updated Power detection
Parts:
- C13: value CP -> 2000uF
- C9: value C -> 0.47uF 450V AC 15mm Pitch; footprint (none) -> Capacitor_THT:CP_Axial_L10.0mm_D6.0mm_P15.00mm_Horizontal
- D2: value DIODE -> DIODE IN4007
- D3: value D_Zener -> 5V_Zener
- R8: value R -> 1k
Changed lines of the file:
@@
 P 1900 5750
 F 0 "C9" V 2152 5750 50  0000 C CNN
-F 1 "C" V 2061 5750 50  0000 C CNN
-F 2 "" H 1938 5600 50  0001 C CNN
+F 1 "0.47uF 450V AC 15mm Pitch" V 2061 5750 50  0000 C CNN
+F 2 "Capacitor_THT:CP_Axial_L10.0mm_D6.0mm_P15.00mm_Horizontal" H 1938 5600 50  0001 C CNN
 F 3 "~" H 1900 5750 50  0001 C CNN
 	1    1900 5750
@@
 P 2450 5750
 F 0 "D2" H 2450 6015 50  0000 C CNN
-F 1 "DIODE" H 2450 5924 50  0000 C CNN
+F 1 "DIODE IN4007" H 2450 5924 50  0000 C CNN
 F 2 "Diode_THT:D_DO-41_SOD81_P10.16mm_Horizontal" H 2450 5750 50  0001 C CNN
 F 3 "~" H 2450 5750 50  0001 C CNN
@@
 P 2750 6100
 F 0 "C13" H 2868 6146 50  0000 L CNN
-F 1 "CP" H 2868 6055 50  0000 L CNN
+F 1 "2000uF" H 2868 6055 50  0000 L CNN
 F 2 "" H 2788 5950 50  0001 C CNN
 F 3 "~" H 2750 6100 50  0001 C CNN
@@
 P 3100 6100
 F 0 "D3" V 3054 6180 50  0000 L CNN
-F 1 "D_Zener" V 3145 6180 50  0000 L CNN
+F 1 "5V_Zener" V 3145 6180 50  0000 L CNN
 F 2 "" H 3100 6100 50  0001 C CNN
 F 3 "~" H 3100 6100 50  0001 C CNN
@@
 P 4600 5750
 F 0 "R8" H 4670 5796 50  0000 L CNN
-F 1 "R" H 4670 5705 50  0000 L CNN
+F 1 "1k" H 4670 5705 50  0000 L CNN
 F 2 "Resistor_SMD:R_0603_1608Metric" V 4530 5750 50  0001 C CNN
 F 3 "~" H 4600 5750 50  0001 C CNN

Commit message: Updated the PCB with component foot prints.
Parts:
- C13: footprint (none) -> Capacitor_THT:CP_Radial_D10.0mm_P2.50mm
- D3: footprint (none) -> Diode_THT:D_DO-35_SOD27_P7.62mm_Horizontal
- H1, H2, H3, H4: footprint MountingHole:MountingHole_4mm -> MountingHole:MountingHole_3.2mm_M3_DIN965_Pad
- J1: footprint Connector_PinHeader_2.54mm:PinHeader_1x02_P2.54mm_Vertical -> TerminalBlock_Phoenix:TerminalBlock_Phoenix_MKDS-1,5-2_1x02_P5.00mm_Horizontal
- J3: footprint (none) -> Connector_BarrelJack:BarrelJack_Horizontal
- J5: footprint (none) -> TerminalBlock_Phoenix:TerminalBlock_Phoenix_MKDS-1,5-2_1x02_P5.00mm_Horizontal
- RV1: footprint (none) -> Varistor:RV_Disc_D21.5mm_W4.4mm_P10mm
- U4: value NSL-32 -> EL814; symbol Isolator:NSL-32 -> Isolator:EL814
Changed lines of the file:
@@
 F 0 "J1" H 4568 1675 50  0000 C CNN
 F 1 "12V INPUT" H 4568 1766 50  0000 C CNN
-F 2 "Connector_PinHeader_2.54mm:PinHeader_1x02_P2.54mm_Vertical" H 4650 2000 50  0001 C CNN
+F 2 "TerminalBlock_Phoenix:TerminalBlock_Phoenix_MKDS-1,5-2_1x02_P5.00mm_Horizontal" H 4650 2000 50  0001 C CNN
 F 3 "~" H 4650 2000 50  0001 C CNN
 	1    4650 2000
@@
 F 0 "H1" H 8250 1496 50  0000 L CNN
 F 1 "MountingHole" H 8250 1405 50  0000 L CNN
-F 2 "MountingHole:MountingHole_4mm" H 8150 1450 50  0001 C CNN
+F 2 "MountingHole:MountingHole_3.2mm_M3_DIN965_Pad" H 8150 1450 50  0001 C CNN
 F 3 "~" H 8150 1450 50  0001 C CNN
 	1    8150 1450
@@
 F 0 "H2" H 8950 1496 50  0000 L CNN
 F 1 "MountingHole" H 8950 1405 50  0000 L CNN
-F 2 "MountingHole:MountingHole_4mm" H 8850 1450 50  0001 C CNN
+F 2 "MountingHole:MountingHole_3.2mm_M3_DIN965_Pad" H 8850 1450 50  0001 C CNN
 F 3 "~" H 8850 1450 50  0001 C CNN
 	1    8850 1450
@@
 F 0 "H3" H 9650 1496 50  0000 L CNN
 F 1 "MountingHole" H 9650 1405 50  0000 L CNN
-F 2 "MountingHole:MountingHole_4mm" H 9550 1450 50  0001 C CNN
+F 2 "MountingHole:MountingHole_3.2mm_M3_DIN965_Pad" H 9550 1450 50  0001 C CNN
 F 3 "~" H 9550 1450 50  0001 C CNN
 	1    9550 1450
@@
 F 0 "H4" H 10350 1496 50  0000 L CNN
 F 1 "MountingHole" H 10350 1405 50  0000 L CNN
-F 2 "MountingHole:MountingHole_4mm" H 10250 1450 50  0001 C CNN
+F 2 "MountingHole:MountingHole_3.2mm_M3_DIN965_Pad" H 10250 1450 50  0001 C CNN
 F 3 "~" H 10250 1450 50  0001 C CNN
 	1    10250 1450
@@
 F 0 "J3" H 6120 1408 50  0000 R CNN
 F 1 "Barrel_Jack" H 6120 1499 50  0000 R CNN
-F 2 "" H 6400 1410 50  0001 C CNN
+F 2 "Connector_BarrelJack:BarrelJack_Horizontal" H 6400 1410 50  0001 C CNN
 F 3 "~" H 6400 1410 50  0001 C CNN
 	1    6350 1450
@@
 F 0 "J5" H 818 5775 50  0000 C CNN
 F 1 "AC INPUT" H 818 5866 50  0000 C CNN
-F 2 "" H 900 6100 50  0001 C CNN
+F 2 "TerminalBlock_Phoenix:TerminalBlock_Phoenix_MKDS-1,5-2_1x02_P5.00mm_Horizontal" H 900 6100 50  0001 C CNN
 F 3 "~" H 900 6100 50  0001 C CNN
 	1    900  6100
@@
 F 0 "RV1" H 1353 6096 50  0000 L CNN
 F 1 "Varistor" H 1353 6005 50  0000 L CNN
-F 2 "" V 1180 6050 50  0001 C CNN
+F 2 "Varistor:RV_Disc_D21.5mm_W4.4mm_P10mm" V 1180 6050 50  0001 C CNN
 F 3 "~" H 1250 6050 50  0001 C CNN
 	1    1250 6050
@@
 F 0 "C13" H 2868 6146 50  0000 L CNN
 F 1 "2000uF" H 2868 6055 50  0000 L CNN
-F 2 "" H 2788 5950 50  0001 C CNN
+F 2 "Capacitor_THT:CP_Radial_D10.0mm_P2.50mm" H 2788 5950 50  0001 C CNN
 F 3 "~" H 2750 6100 50  0001 C CNN
 	1    2750 6100
@@
 F 0 "D3" V 3054 6180 50  0000 L CNN
 F 1 "5V_Zener" V 3145 6180 50  0000 L CNN
-F 2 "" H 3100 6100 50  0001 C CNN
+F 2 "Diode_THT:D_DO-35_SOD27_P7.62mm_Horizontal" H 3100 6100 50  0001 C CNN
 F 3 "~" H 3100 6100 50  0001 C CNN
 	1    3100 6100
@@
 $EndComp
 $Comp
-L Isolator:NSL-32 U4
+L Isolator:EL814 U4
 U 1 1 606D3219
 P 4100 6100
 F 0 "U4" H 4100 6417 50  0000 C CNN
-F 1 "NSL-32" H 4100 6326 50  0000 C CNN
+F 1 "EL814" H 4100 6326 50  0000 C CNN
 F 2 "OptoDevice:Luna_NSL-32" H 4100 5800 50  0001 C CNN
 F 3 "http://lunainc.com/wp-content/uploads/2016/06/NSL-32.pdf" H 4150 6100 50  0001 C CNN

Commit message: updated the platform PCB.
Parts:
- C13: value 2000uF -> 1000uF
- C9: footprint Capacitor_THT:CP_Axial_L10.0mm_D6.0mm_P15.00mm_Horizontal -> Capacitor_THT:C_Rect_L7.2mm_W5.5mm_P5.00mm_FKS2_FKP2_MKS2_MKP2
- J8: footprint Connector_PinHeader_2.54mm:PinHeader_1x06_P2.54mm_Vertical -> Connector_Molex:Molex_KK-254_AE-6410-06A_1x06_P2.54mm_Vertical
- R5: value R -> 470K 1W; footprint Resistor_SMD:R_0603_1608Metric -> Resistor_THT:R_Axial_DIN0411_L9.9mm_D3.6mm_P12.70mm_Horizontal
- R6: value R -> 100E 1W; footprint Resistor_SMD:R_0603_1608Metric -> Resistor_THT:R_Axial_DIN0411_L9.9mm_D3.6mm_P12.70mm_Horizontal
- R7: value R -> 220E
- RV1: footprint Varistor:RV_Disc_D21.5mm_W4.4mm_P10mm -> Varistor:RV_Disc_D7mm_W3.4mm_P5mm
Changed lines of the file:
@@
-$EndComp
-$Comp
-L power:GND #PWR08
-U 1 1 5FABFC8F
-P 8150 1500
-F 0 "#PWR08" H 8150 1250 50  0001 C CNN
-F 1 "GND" H 8155 1327 50  0000 C CNN
-F 2 "" H 8150 1500 50  0001 C CNN
-F 3 "" H 8150 1500 50  0001 C CNN
-	1    8150 1500
-	1    0    0    -1
 $EndComp
 $Comp
@@
 F 0 "J8" H 2730 3592 50  0000 L CNN
 F 1 "Conn_01x06" H 2730 3501 50  0000 L CNN
-F 2 "Connector_PinHeader_2.54mm:PinHeader_1x06_P2.54mm_Vertical" H 2650 3600 50  0001 C CNN
+F 2 "Connector_Molex:Molex_KK-254_AE-6410-06A_1x06_P2.54mm_Vertical" H 2650 3600 50  0001 C CNN
 F 3 "~" H 2650 3600 50  0001 C CNN
 	1    2650 3600
@@
 F 0 "RV1" H 1353 6096 50  0000 L CNN
 F 1 "Varistor" H 1353 6005 50  0000 L CNN
-F 2 "Varistor:RV_Disc_D21.5mm_W4.4mm_P10mm" V 1180 6050 50  0001 C CNN
+F 2 "Varistor:RV_Disc_D7mm_W3.4mm_P5mm" V 1180 6050 50  0001 C CNN
 F 3 "~" H 1250 6050 50  0001 C CNN
 	1    1250 6050
@@
 F 0 "C9" V 2152 5750 50  0000 C CNN
 F 1 "0.47uF 450V AC 15mm Pitch" V 2061 5750 50  0000 C CNN
-F 2 "Capacitor_THT:CP_Axial_L10.0mm_D6.0mm_P15.00mm_Horizontal" H 1938 5600 50  0001 C CNN
+F 2 "Capacitor_THT:C_Rect_L7.2mm_W5.5mm_P5.00mm_FKS2_FKP2_MKS2_MKP2" H 1938 5600 50  0001 C CNN
 F 3 "~" H 1900 5750 50  0001 C CNN
 	1    1900 5750
@@
 P 1900 6100
 F 0 "R5" V 1693 6100 50  0000 C CNN
-F 1 "R" V 1784 6100 50  0000 C CNN
-F 2 "Resistor_SMD:R_0603_1608Metric" V 1830 6100 50  0001 C CNN
+F 1 "470K 1W" V 1784 6100 50  0000 C CNN
+F 2 "Resistor_THT:R_Axial_DIN0411_L9.9mm_D3.6mm_P12.70mm_Horizontal" V 1830 6100 50  0001 C CNN
 F 3 "~" H 1900 6100 50  0001 C CNN
 	1    1900 6100
@@
 P 1900 6550
 F 0 "R6" V 1693 6550 50  0000 C CNN
-F 1 "R" V 1784 6550 50  0000 C CNN
-F 2 "Resistor_SMD:R_0603_1608Metric" V 1830 6550 50  0001 C CNN
+F 1 "100E 1W" V 1784 6550 50  0000 C CNN
+F 2 "Resistor_THT:R_Axial_DIN0411_L9.9mm_D3.6mm_P12.70mm_Horizontal" V 1830 6550 50  0001 C CNN
 F 3 "~" H 1900 6550 50  0001 C CNN
 	1    1900 6550
@@
 P 2750 6100
 F 0 "C13" H 2868 6146 50  0000 L CNN
-F 1 "2000uF" H 2868 6055 50  0000 L CNN
+F 1 "1000uF" H 2868 6055 50  0000 L CNN
 F 2 "Capacitor_THT:CP_Radial_D10.0mm_P2.50mm" H 2788 5950 50  0001 C CNN
 F 3 "~" H 2750 6100 50  0001 C CNN
@@
 P 3450 5750
 F 0 "R7" V 3243 5750 50  0000 C CNN
-F 1 "R" V 3334 5750 50  0000 C CNN
+F 1 "220E" V 3334 5750 50  0000 C CNN
 F 2 "Resistor_SMD:R_0603_1608Metric" V 3380 5750 50  0001 C CNN
 F 3 "~" H 3450 5750 50  0001 C CNN

Commit message: Updated component values.
Parts:
- R2: value 5.1K -> 1.65K
Changed lines of the file:
@@
 P 7850 5250
 F 0 "R2" H 7920 5296 50  0000 L CNN
-F 1 "5.1K" H 7920 5205 50  0000 L CNN
+F 1 "1.65K" H 7920 5205 50  0000 L CNN
 F 2 "Resistor_SMD:R_0603_1608Metric" V 7780 5250 50  0001 C CNN
 F 3 "~" H 7850 5250 50  0001 C CNN
