File: Platform/MCU.sch (KiCad schematic (older format))
At the start: 24 parts, among them J10 Conn_01x05, J12 Aardvark Header I2C, J13 ESP8266_CONN, J14 Aardvark Header I2C/SPI, J4 Conn_01x05, J6 Debug Hdr, J7 Conn_01x05, U3 ATSAMD21E16B-M

Commit message: Added connector for relay controls.
Parts:
- added J11: Relay_conn, symbol Connector_Generic:Conn_01x04
- C6, C7, C8: symbol Device:CP -> Device:C
- R11, R12, R13, R14, R17, R18, R19, R20, R21, R3, R4: footprint (none) -> Resistor_SMD:R_0603_1608Metric
- gave numbers to parts that had none: 1
Connections:
- net GND: now also J11.4 (Pin_4)
- net PA16: now also J11.1 (Pin_1)
- net PA17: now also J11.2 (Pin_2)
- net PA18: now also J11.3 (Pin_3)
Other:
- note added: "Relay Controls"
Changed lines of the file:
@@
 F 0 "R3" H 3270 3896 50  0000 L CNN
 F 1 "10K" H 3270 3805 50  0000 L CNN
-F 2 "" V 3130 3850 50  0001 C CNN
+F 2 "Resistor_SMD:R_0603_1608Metric" V 3130 3850 50  0001 C CNN
 F 3 "~" H 3200 3850 50  0001 C CNN
 	1    3200 3850
@@
 F 0 "R11" H 8170 2746 50  0000 L CNN
 F 1 "1K DNP" H 8170 2655 50  0000 L CNN
-F 2 "" V 8030 2700 50  0001 C CNN
+F 2 "Resistor_SMD:R_0603_1608Metric" V 8030 2700 50  0001 C CNN
 F 3 "~" H 8100 2700 50  0001 C CNN
 	1    8100 2700
@@
 F 0 "R12" H 8070 2746 50  0000 L CNN
 F 1 "1K DNP" H 8070 2655 50  0000 L CNN
-F 2 "" V 7930 2700 50  0001 C CNN
+F 2 "Resistor_SMD:R_0603_1608Metric" V 7930 2700 50  0001 C CNN
 F 3 "~" H 8000 2700 50  0001 C CNN
 	1    8000 2700
@@
 	7350 4000 7350 2300
 $Comp
-L Device:CP C7
+L Device:C C7
 U 1 1 5FB646A0
 P 4900 1400
@@
 $EndComp
 $Comp
-L Device:CP C6
+L Device:C C6
 U 1 1 5FB67AB7
 P 4250 1400
@@
 $EndComp
 $Comp
-L Device:CP C8
+L Device:C C8
 U 1 1 5FB6BF77
 P 6600 1600
@@
 F 0 "R4" H 1770 4396 50  0000 L CNN
 F 1 "1K" H 1770 4305 50  0000 L CNN
-F 2 "" V 1630 4350 50  0001 C CNN
+F 2 "Resistor_SMD:R_0603_1608Metric" V 1630 4350 50  0001 C CNN
 F 3 "~" H 1700 4350 50  0001 C CNN
 	1    1700 4350
@@
 F 0 "R18" V 9193 4950 50  0000 C CNN
 F 1 "1K" V 9284 4950 50  0000 C CNN
-F 2 "" V 9330 4950 50  0001 C CNN
+F 2 "Resistor_SMD:R_0603_1608Metric" V 9330 4950 50  0001 C CNN
 F 3 "~" H 9400 4950 50  0001 C CNN
 	1    9400 4950
@@
 F 0 "R17" V 8943 3150 50  0000 C CNN
 F 1 "0 DNP" V 9034 3150 50  0000 C CNN
-F 2 "" V 9080 3150 50  0001 C CNN
+F 2 "Resistor_SMD:R_0603_1608Metric" V 9080 3150 50  0001 C CNN
 F 3 "~" H 9150 3150 50  0001 C CNN
 	1    9150 3150
@@
 F 0 "R19" V 10057 3250 50  0000 C CNN
 F 1 "0 DNP" V 9966 3250 50  0000 C CNN
-F 2 "" V 9780 3250 50  0001 C CNN
+F 2 "Resistor_SMD:R_0603_1608Metric" V 9780 3250 50  0001 C CNN
 F 3 "~" H 9850 3250 50  0001 C CNN
 	1    9850 3250
@@
 F 0 "R20" V 9793 1500 50  0000 C CNN
 F 1 "0 DNP" V 9884 1500 50  0000 C CNN
-F 2 "" V 9930 1500 50  0001 C CNN
+F 2 "Resistor_SMD:R_0603_1608Metric" V 9930 1500 50  0001 C CNN
 F 3 "~" H 10000 1500 50  0001 C CNN
 	1    10000 1500
@@
 F 0 "R21" V 10857 1700 50  0000 C CNN
 F 1 "0 DNP" V 10766 1700 50  0000 C CNN
-F 2 "" V 10580 1700 50  0001 C CNN
+F 2 "Resistor_SMD:R_0603_1608Metric" V 10580 1700 50  0001 C CNN
 F 3 "~" H 10650 1700 50  0001 C CNN
 	1    10650 1700
@@
 F 0 "R14" H 8959 1296 50  0000 L CNN
 F 1 "R_Small" H 8959 1205 50  0000 L CNN
-F 2 "" H 8900 1250 50  0001 C CNN
+F 2 "Resistor_SMD:R_0603_1608Metric" H 8900 1250 50  0001 C CNN
 F 3 "~" H 8900 1250 50  0001 C CNN
 	1    8900 1250
@@
 F 0 "R13" H 8741 1204 50  0000 R CNN
 F 1 "R_Small" H 8741 1295 50  0000 R CNN
-F 2 "" H 8800 1250 50  0001 C CNN
+F 2 "Resistor_SMD:R_0603_1608Metric" H 8800 1250 50  0001 C CNN
 F 3 "~" H 8800 1250 50  0001 C CNN
 	1    8800 1250
@@
 	550  5700 4150 5700
 $Comp
-L Connector_Generic:Conn_02x10_Odd_Even J?
+L Connector_Generic:Conn_02x10_Odd_Even J9
 U 1 1 6069055C
 P 2150 2150
-F 0 "J?" H 2200 2767 50  0000 C CNN
+F 0 "J9" H 2200 2767 50  0000 C CNN
 F 1 "LED Interface" H 2200 2676 50  0000 C CNN
 F 2 "" H 2150 2150 50  0001 C CNN
@@
 	2600 1850 2450 1850
 $Comp
-L power:GND #PWR?
+L power:GND #PWR041
 U 1 1 606D565B
 P 2600 2750
-F 0 "#PWR?" H 2600 2500 50  0001 C CNN
+F 0 "#PWR041" H 2600 2500 50  0001 C CNN
 F 1 "GND" H 2605 2577 50  0000 C CNN
 F 2 "" H 2600 2750 50  0001 C CNN
@@
 $EndComp
 $Comp
-L power:GND #PWR?
+L power:GND #PWR029
 U 1 1 606D5B76
 P 1800 2750
-F 0 "#PWR?" H 1800 2500 50  0001 C CNN
+F 0 "#PWR029" H 1800 2500 50  0001 C CNN
 F 1 "GND" H 1805 2577 50  0000 C CNN
 F 2 "" H 1800 2750 50  0001 C CNN
@@
 	1800 2650 1950 2650
 $Comp
-L power:+5V #PWR?
+L power:+5V #PWR032
 U 1 1 606DFE5F
 P 2600 1550
-F 0 "#PWR?" H 2600 1400 50  0001 C CNN
+F 0 "#PWR032" H 2600 1400 50  0001 C CNN
 F 1 "+5V" V 2615 1678 50  0000 L CNN
 F 2 "" H 2600 1550 50  0001 C CNN
@@
 $EndComp
 $Comp
-L power:+5V #PWR?
+L power:+5V #PWR026
 U 1 1 606E0CFA
 P 1800 1550
-F 0 "#PWR?" H 1800 1400 50  0001 C CNN
+F 0 "#PWR026" H 1800 1400 50  0001 C CNN
 F 1 "+5V" V 1815 1678 50  0000 L CNN
 F 2 "" H 1800 1550 50  0001 C CNN
@@
 Text Notes 1600 3150 0    50   ~ 0
 MCU-LED interface connector
+$Comp
+L Connector_Generic:Conn_01x04 J11
+U 1 1 606AD8C9
+P 5600 6450
+F 0 "J11" H 5680 6442 50  0000 L CNN
+F 1 "Relay_conn" H 5680 6351 50  0000 L CNN
+F 2 "" H 5600 6450 50  0001 C CNN
+F 3 "~" H 5600 6450 50  0001 C CNN
+	1    5600 6450
+	1    0    0    -1
+$EndComp
+$Comp
+L power:GND #PWR042
+U 1 1 606B0151
+P 5250 6750
+F 0 "#PWR042" H 5250 6500 50  0001 C CNN
+F 1 "GND" H 5255 6577 50  0000 C CNN
+F 2 "" H 5250 6750 50  0001 C CNN
+F 3 "" H 5250 6750 50  0001 C CNN
+	1    5250 6750
+	1    0    0    -1
+$EndComp
+Wire Wire Line
+	5250 6750 5250 6650
+Wire Wire Line
+	5250 6650 5400 6650
+Text GLabel 5250 6550 0    50   BiDi ~ 10
+PA18
+Text GLabel 5250 6450 0    50   BiDi ~ 10
+PA17
+Text GLabel 5250 6350 0    50   BiDi ~ 10
+PA16
+Wire Wire Line
+	5250 6350 5400 6350
+Wire Wire Line
+	5400 6450 5250 6450
+Wire Wire Line
+	5250 6550 5400 6550
+Wire Notes Line
+	6300 6150 6300 7350
+Wire Notes Line
+	6300 7350 4600 7350
+Wire Notes Line
+	4600 7350 4600 6150
+Wire Notes Line
+	4600 6150 6300 6150
+Text Notes 5000 7200 0    50   ~ 0
+Relay Controls
 $EndSCHEMATC

Commit message: updated.
Parts:
- J10, J7: footprint (none) -> Connector_PinHeader_2.54mm:PinHeader_1x05_P2.54mm_Vertical
- J11: footprint (none) -> Connector_PinHeader_2.54mm:PinHeader_1x04_P2.54mm_Vertical
- J12: footprint (none) -> Connector_PinHeader_2.54mm:PinHeader_2x05_P2.54mm_Vertical
- J13: footprint (none) -> Connector_PinHeader_2.54mm:PinHeader_2x04_P2.54mm_Vertical
- J9: footprint (none) -> Connector_PinHeader_2.54mm:PinHeader_2x10_P2.54mm_Horizontal
Changed lines of the file:
@@
 F 0 "J12" H 8500 3667 50  0000 C CNN
 F 1 "Aardvark Header I2C" H 8500 3576 50  0000 C CNB
-F 2 "" H 8450 3250 50  0001 C CNN
+F 2 "Connector_PinHeader_2.54mm:PinHeader_2x05_P2.54mm_Vertical" H 8450 3250 50  0001 C CNN
 F 3 "~" H 8450 3250 50  0001 C CNN
 	1    8450 3250
@@
 F 0 "J13" H 8550 5167 50  0000 C CNN
 F 1 "ESP8266_CONN" H 8550 5076 50  0000 C CNN
-F 2 "" H 8500 4850 50  0001 C CNN
+F 2 "Connector_PinHeader_2.54mm:PinHeader_2x04_P2.54mm_Vertical" H 8500 4850 50  0001 C CNN
 F 3 "~" H 8500 4850 50  0001 C CNN
 	1    8500 4850
@@
 F 0 "J7" H 2480 6092 50  0000 L CNN
 F 1 "Conn_01x05" H 2480 6001 50  0000 L CNN
-F 2 "" H 2400 6050 50  0001 C CNN
+F 2 "Connector_PinHeader_2.54mm:PinHeader_1x05_P2.54mm_Vertical" H 2400 6050 50  0001 C CNN
 F 3 "~" H 2400 6050 50  0001 C CNN
 	1    2400 6050
@@
 F 0 "J10" H 3580 6092 50  0000 L CNN
 F 1 "Conn_01x05" H 3580 6001 50  0000 L CNN
-F 2 "" H 3500 6050 50  0001 C CNN
+F 2 "Connector_PinHeader_2.54mm:PinHeader_1x05_P2.54mm_Vertical" H 3500 6050 50  0001 C CNN
 F 3 "~" H 3500 6050 50  0001 C CNN
 	1    3500 6050
@@
 F 0 "J9" H 2200 2767 50  0000 C CNN
 F 1 "LED Interface" H 2200 2676 50  0000 C CNN
-F 2 "" H 2150 2150 50  0001 C CNN
+F 2 "Connector_PinHeader_2.54mm:PinHeader_2x10_P2.54mm_Horizontal" H 2150 2150 50  0001 C CNN
 F 3 "~" H 2150 2150 50  0001 C CNN
 	1    2150 2150
@@
 F 0 "J11" H 5680 6442 50  0000 L CNN
 F 1 "Relay_conn" H 5680 6351 50  0000 L CNN
-F 2 "" H 5600 6450 50  0001 C CNN
+F 2 "Connector_PinHeader_2.54mm:PinHeader_1x04_P2.54mm_Vertical" H 5600 6450 50  0001 C CNN
 F 3 "~" H 5600 6450 50  0001 C CNN
 	1    5600 6450
