File: Platform/MCU.sch (KiCad schematic (older format))
At the start: 25 parts, among them J10 Conn_01x05, J11 Relay_conn, J12 Aardvark Header I2C, J13 ESP8266_CONN, J14 Aardvark Header I2C/SPI, J4 Conn_01x05, J6 Debug Hdr, J7 Conn_01x05, J9 LED Interface, U3 ATSAMD21E16B-M

Commit message: GRM155R61C105KE01D
Parts:
- C6, C7, C8: footprint (none) -> Capacitor_SMD:C_0402_1005Metric
- J14, J6: footprint (none) -> Connector_PinHeader_2.54mm:PinHeader_2x05_P2.54mm_Vertical
- J4: footprint (none) -> Connector_PinHeader_2.54mm:PinHeader_1x05_P2.54mm_Vertical
- U3: symbol Platform-rescue:ATSAMD21E16B-M-MCU_Microchip_SAMD-Platform-rescue -> Platform-rescue:ATSAMD21E16B-M-MCU_Microchip_SAMD-Platform-rescue-Platform-rescue
Changed lines of the file:
@@
 F 0 "J6" H 1400 5167 50  0000 C CNN
 F 1 "Debug Hdr" H 1400 5076 50  0000 C CNN
-F 2 "" H 1350 4750 50  0001 C CNN
+F 2 "Connector_PinHeader_2.54mm:PinHeader_2x05_P2.54mm_Vertical" H 1350 4750 50  0001 C CNN
 F 3 "~" H 1350 4750 50  0001 C CNN
 	1    1350 4750
@@
 RESET
 $Comp
-L Platform-rescue:ATSAMD21E16B-M-MCU_Microchip_SAMD-Platform-rescue U3
+L Platform-rescue:ATSAMD21E16B-M-MCU_Microchip_SAMD-Platform-rescue-Platform-rescue U3
 U 1 1 5FAA26F4
 P 5700 3450
@@
 F 0 "J14" H 9400 2017 50  0000 C CNN
 F 1 "Aardvark Header I2C/SPI" H 9600 2100 50  0000 C CNB
-F 2 "" H 9350 1600 50  0001 C CNN
+F 2 "Connector_PinHeader_2.54mm:PinHeader_2x05_P2.54mm_Vertical" H 9350 1600 50  0001 C CNN
 F 3 "~" H 9350 1600 50  0001 C CNN
 	1    9350 1600
@@
 F 0 "C7" H 5018 1446 50  0000 L CNN
 F 1 "1uF" H 5018 1355 50  0000 L CNN
-F 2 "" H 4938 1250 50  0001 C CNN
+F 2 "Capacitor_SMD:C_0402_1005Metric" H 4938 1250 50  0001 C CNN
 F 3 "~" H 4900 1400 50  0001 C CNN
 	1    4900 1400
@@
 F 0 "C6" H 4368 1446 50  0000 L CNN
 F 1 "100nF DNP" H 4368 1355 50  0000 L CNN
-F 2 "" H 4288 1250 50  0001 C CNN
+F 2 "Capacitor_SMD:C_0402_1005Metric" H 4288 1250 50  0001 C CNN
 F 3 "~" H 4250 1400 50  0001 C CNN
 	1    4250 1400
@@
 F 0 "C8" H 6718 1646 50  0000 L CNN
 F 1 "100nF DNP" H 6718 1555 50  0000 L CNN
-F 2 "" H 6638 1450 50  0001 C CNN
+F 2 "Capacitor_SMD:C_0402_1005Metric" H 6638 1450 50  0001 C CNN
 F 3 "~" H 6600 1600 50  0001 C CNN
 	1    6600 1600
@@
 F 0 "J4" H 1380 6092 50  0000 L CNN
 F 1 "Conn_01x05" H 1380 6001 50  0000 L CNN
-F 2 "" H 1300 6050 50  0001 C CNN
+F 2 "Connector_PinHeader_2.54mm:PinHeader_1x05_P2.54mm_Vertical" H 1300 6050 50  0001 C CNN
 F 3 "~" H 1300 6050 50  0001 C CNN
 	1    1300 6050

Commit message: Updated the PCB with component foot prints.
Parts:
- C14: footprint (none) -> Capacitor_SMD:C_0402_1005Metric
Changed lines of the file:
@@
 F 0 "C14" H 3292 4446 50  0000 L CNN
 F 1 "C_Small" H 3292 4355 50  0000 L CNN
-F 2 "" H 3200 4400 50  0001 C CNN
+F 2 "Capacitor_SMD:C_0402_1005Metric" H 3200 4400 50  0001 C CNN
 F 3 "~" H 3200 4400 50  0001 C CNN
 	1    3200 4400

Commit message: updated the platform PCB.
Parts:
- J11: footprint Connector_PinHeader_2.54mm:PinHeader_1x04_P2.54mm_Vertical -> Connector_Molex:Molex_KK-254_AE-6410-04A_1x04_P2.54mm_Vertical
Changed lines of the file:
@@
 F 0 "J11" H 5680 6442 50  0000 L CNN
 F 1 "Relay_conn" H 5680 6351 50  0000 L CNN
-F 2 "Connector_PinHeader_2.54mm:PinHeader_1x04_P2.54mm_Vertical" H 5600 6450 50  0001 C CNN
+F 2 "Connector_Molex:Molex_KK-254_AE-6410-04A_1x04_P2.54mm_Vertical" H 5600 6450 50  0001 C CNN
 F 3 "~" H 5600 6450 50  0001 C CNN
 	1    5600 6450
