File: Platform/RTC_EEPROM.sch (KiCad schematic (older format))
At the start: 15 parts, among them U5 AT24CS32-SSHM, U6 MCP7940N-xMS, Y1 32KHz crystal

Commit message: Added power input detection circuit.
Parts:
- gave numbers to parts that had none: 1
Changed lines of the file:
@@
 	8150 2350 8450 2350
 $Comp
-L Connector:TestPoint TP?
+L Connector:TestPoint TP1
 U 1 1 60677E6E
 P 5350 2450
-F 0 "TP?" V 5545 2522 50  0000 C CNN
+F 0 "TP1" V 5545 2522 50  0000 C CNN
 F 1 "TestPoint" V 5454 2522 50  0000 C CNN
 F 2 "" H 5550 2450 50  0001 C CNN

Commit message: Added connector for relay controls.
Parts:
- BAT1: footprint digikey-footprints:Battery_Holder_Coin_2032_BS-7 -> Battery:BatteryHolder_Keystone_103_1x20mm
- C10: symbol Device:CP -> Device:C
- R25, R26, R27, R28, R29, R30, R31: footprint (none) -> Resistor_SMD:R_0603_1608Metric
- Y1: footprint (none) -> Crystal:Crystal_AT310_D3.0mm_L10.0mm_Horizontal_1EP_style2; symbol Device:Crystal_GND2 -> Device:Crystal_GND3
Connections:
- net labels removed: VBAT
- wire segments 67 -> 65
Changed lines of the file:
@@
 F 0 "BAT1" H 7628 1703 60  0000 L CNN
 F 1 "BS-7    3.3V" H 7628 1597 60  0000 L CNN
-F 2 "digikey-footprints:Battery_Holder_Coin_2032_BS-7" H 7700 1850 60  0001 L CNN
+F 2 "Battery:BatteryHolder_Keystone_103_1x20mm" H 7700 1850 60  0001 L CNN
 F 3 "http://www.memoryprotectiondevices.com/datasheets/BS-7-datasheet.pdf" V 7700 1950 60  0001 L CNN
 F 4 "BS-7-ND" H 7700 2050 60  0001 L CNN "Digi-Key_PN"
@@
 $EndComp
 $Comp
-L Device:CP C10
+L Device:C C10
 U 1 1 5FB42048
 P 5350 1800
@@
 L power:GND #PWR052
 U 1 1 5FB45567
-P 7800 1850
-F 0 "#PWR052" H 7800 1600 50  0001 C CNN
-F 1 "GND" H 7805 1677 50  0000 C CNN
-F 2 "" H 7800 1850 50  0001 C CNN
-F 3 "" H 7800 1850 50  0001 C CNN
-	1    7800 1850
+P 7500 1900
+F 0 "#PWR052" H 7500 1650 50  0001 C CNN
+F 1 "GND" H 7505 1727 50  0000 C CNN
+F 2 "" H 7500 1900 50  0001 C CNN
+F 3 "" H 7500 1900 50  0001 C CNN
+	1    7500 1900
 	1    0    0    -1
 $EndComp
@@
 F 0 "R27" H 6220 1846 50  0000 L CNN
 F 1 "2K" H 6220 1755 50  0000 L CNN
-F 2 "" V 6080 1800 50  0001 C CNN
+F 2 "Resistor_SMD:R_0603_1608Metric" V 6080 1800 50  0001 C CNN
 F 3 "~" H 6150 1800 50  0001 C CNN
 	1    6150 1800
@@
 F 0 "R26" H 5820 1846 50  0000 L CNN
 F 1 "2K" H 5820 1755 50  0000 L CNN
-F 2 "" V 5680 1800 50  0001 C CNN
+F 2 "Resistor_SMD:R_0603_1608Metric" V 5680 1800 50  0001 C CNN
 F 3 "~" H 5750 1800 50  0001 C CNN
 	1    5750 1800
@@
 F 0 "R25" H 5670 2246 50  0000 L CNN
 F 1 "10K" H 5670 2155 50  0000 L CNN
-F 2 "" V 5530 2200 50  0001 C CNN
+F 2 "Resistor_SMD:R_0603_1608Metric" V 5530 2200 50  0001 C CNN
 F 3 "~" H 5600 2200 50  0001 C CNN
 	1    5600 2200
@@
 F 0 "R28" H 6970 5046 50  0000 L CNN
 F 1 "2K" H 6970 4955 50  0000 L CNN
-F 2 "" V 6830 5000 50  0001 C CNN
+F 2 "Resistor_SMD:R_0603_1608Metric" V 6830 5000 50  0001 C CNN
 F 3 "~" H 6900 5000 50  0001 C CNN
 	1    6900 5000
@@
 F 0 "R29" H 7370 5146 50  0000 L CNN
 F 1 "2K" H 7370 5055 50  0000 L CNN
-F 2 "" V 7230 5100 50  0001 C CNN
+F 2 "Resistor_SMD:R_0603_1608Metric" V 7230 5100 50  0001 C CNN
 F 3 "~" H 7300 5100 50  0001 C CNN
 	1    7300 5100
@@
 	7150 1450 7500 1450
 Wire Wire Line
-	7800 1850 7500 1850
+	7500 1900 7500 1850
 $Comp
 L Device:R_Small R30
@@
 F 0 "R30" V 1650 600 50  0000 C CNN
 F 1 "0E" V 1750 700 50  0000 C CNN
-F 2 "" H 1700 700 50  0001 C CNN
+F 2 "Resistor_SMD:R_0603_1608Metric" H 1700 700 50  0001 C CNN
 F 3 "~" H 1700 700 50  0001 C CNN
 	1    1700 700
@@
 F 0 "R31" V 1650 800 50  0000 C CNN
 F 1 "0E" V 1800 900 50  0000 C CNN
-F 2 "" H 1700 900 50  0001 C CNN
+F 2 "Resistor_SMD:R_0603_1608Metric" H 1700 900 50  0001 C CNN
 F 3 "~" H 1700 900 50  0001 C CNN
 	1    1700 900
@@
 added 0ohm resistors for easy rework.
 $Comp
-L Device:Crystal_GND2 Y1
+L Device:Crystal_GND3 Y1
 U 1 1 5FBAC838
 P 7950 2350
 F 0 "Y1" V 7996 2481 50  0000 L CNN
 F 1 "32KHz crystal" V 8100 1800 50  0000 L CNN
-F 2 "" H 7950 2350 50  0001 C CNN
+F 2 "Crystal:Crystal_AT310_D3.0mm_L10.0mm_Horizontal_1EP_style2" H 7950 2350 50  0001 C CNN
 F 3 "~" H 7950 2350 50  0001 C CNN
 	1    7950 2350
@@
 	1    0    0    -1
 $EndComp
-Text GLabel 7600 1300 2    50   Output ~ 0
-VBAT
-Wire Wire Line
-	7600 1300 7500 1300
-Wire Wire Line
-	7500 1300 7500 1450
-Connection ~ 7500 1450
 $Comp
 L Device:C_Small C11

Commit message: GRM155R61C105KE01D
Parts:
- BAT1: symbol Platform-rescue:BS-7-dk_Battery-Holders-Clips-Contacts-Platform-rescue -> Platform-rescue:BS-7-dk_Battery-Holders-Clips-Contacts-Platform-rescue-Platform-rescue
- C10: footprint (none) -> Capacitor_SMD:C_0402_1005Metric
- TP1: footprint (none) -> TestPoint:TestPoint_THTPad_3.0x3.0mm_Drill1.5mm
- U6: footprint (none) -> Package_SO:SOIC-8_3.9x4.9mm_P1.27mm
Changed lines of the file:
@@
 F 0 "U6" H 7050 1861 50  0000 C CNN
 F 1 "MCP7940N-xMS" H 7050 1770 50  0000 C CNN
-F 2 "" H 7050 2350 50  0001 C CNN
+F 2 "Package_SO:SOIC-8_3.9x4.9mm_P1.27mm" H 7050 2350 50  0001 C CNN
 F 3 "http://ww1.microchip.com/downloads/en/DeviceDoc/20005010F.pdf" H 7050 2350 50  0001 C CNN
 	1    7050 2350
@@
 $EndComp
 $Comp
-L Platform-rescue:BS-7-dk_Battery-Holders-Clips-Contacts-Platform-rescue BAT1
+L Platform-rescue:BS-7-dk_Battery-Holders-Clips-Contacts-Platform-rescue-Platform-rescue BAT1
 U 1 1 5FB40A5C
 P 7500 1650
@@
 F 0 "C10" H 5468 1846 50  0000 L TNN
 F 1 "0.1U to 1UF" H 5468 1755 50  0000 R TNN
-F 2 "" H 5388 1650 50  0001 C CNN
+F 2 "Capacitor_SMD:C_0402_1005Metric" H 5388 1650 50  0001 C CNN
 F 3 "~" H 5350 1800 50  0001 C CNN
 	1    5350 1800
@@
 F 0 "TP1" V 5545 2522 50  0000 C CNN
 F 1 "TestPoint" V 5454 2522 50  0000 C CNN
-F 2 "" H 5550 2450 50  0001 C CNN
+F 2 "TestPoint:TestPoint_THTPad_3.0x3.0mm_Drill1.5mm" H 5550 2450 50  0001 C CNN
 F 3 "~" H 5550 2450 50  0001 C CNN
 	1    5350 2450

Commit message: Updated the PCB with component foot prints.
Parts:
- C11, C12: footprint (none) -> Capacitor_SMD:C_0402_1005Metric
Changed lines of the file:
@@
 F 0 "C11" V 7971 2100 50  0000 C CNN
 F 1 "C_Small" V 8062 2100 50  0000 C CNN
-F 2 "" H 8200 2100 50  0001 C CNN
+F 2 "Capacitor_SMD:C_0402_1005Metric" H 8200 2100 50  0001 C CNN
 F 3 "~" H 8200 2100 50  0001 C CNN
 	1    8200 2100
@@
 F 0 "C12" V 7971 2600 50  0000 C CNN
 F 1 "C_Small" V 8062 2600 50  0000 C CNN
-F 2 "" H 8200 2600 50  0001 C CNN
+F 2 "Capacitor_SMD:C_0402_1005Metric" H 8200 2600 50  0001 C CNN
 F 3 "~" H 8200 2600 50  0001 C CNN
 	1    8200 2600

Commit message: updated the platform PCB.
Parts:
- TP1: footprint TestPoint:TestPoint_THTPad_3.0x3.0mm_Drill1.5mm -> TestPoint:TestPoint_Pad_D2.5mm
Changed lines of the file:
@@
 F 0 "TP1" V 5545 2522 50  0000 C CNN
 F 1 "TestPoint" V 5454 2522 50  0000 C CNN
-F 2 "TestPoint:TestPoint_THTPad_3.0x3.0mm_Drill1.5mm" H 5550 2450 50  0001 C CNN
+F 2 "TestPoint:TestPoint_Pad_D2.5mm" H 5550 2450 50  0001 C CNN
 F 3 "~" H 5550 2450 50  0001 C CNN
 	1    5350 2450
