File: LED_DC/LED_DC/MCU_IF.sch (KiCad schematic (older format))
At the start: 4 parts

Commit message: Updated PCB.
Parts:
- H1, H2, H3, H4: footprint MountingHole:MountingHole_2.2mm_M2_DIN965_Pad -> MountingHole:MountingHole_3.2mm_M3_DIN965_Pad
Changed lines of the file:
@@
 F 0 "H1" H 8400 1503 50  0000 L CNN
 F 1 "MountingHole_Pad" H 8400 1458 50  0001 L CNN
-F 2 "MountingHole:MountingHole_2.2mm_M2_DIN965_Pad" H 8300 1500 50  0001 C CNN
+F 2 "MountingHole:MountingHole_3.2mm_M3_DIN965_Pad" H 8300 1500 50  0001 C CNN
 F 3 "~" H 8300 1500 50  0001 C CNN
 	1    8300 1500
@@
 F 0 "H2" H 8800 1503 50  0000 L CNN
 F 1 "MountingHole_Pad" H 8800 1458 50  0001 L CNN
-F 2 "MountingHole:MountingHole_2.2mm_M2_DIN965_Pad" H 8700 1500 50  0001 C CNN
+F 2 "MountingHole:MountingHole_3.2mm_M3_DIN965_Pad" H 8700 1500 50  0001 C CNN
 F 3 "~" H 8700 1500 50  0001 C CNN
 	1    8700 1500
@@
 F 0 "H3" H 9200 1503 50  0000 L CNN
 F 1 "MountingHole_Pad" H 9200 1458 50  0001 L CNN
-F 2 "MountingHole:MountingHole_2.2mm_M2_DIN965_Pad" H 9100 1500 50  0001 C CNN
+F 2 "MountingHole:MountingHole_3.2mm_M3_DIN965_Pad" H 9100 1500 50  0001 C CNN
 F 3 "~" H 9100 1500 50  0001 C CNN
 	1    9100 1500
@@
 F 0 "H4" H 9550 1503 50  0000 L CNN
 F 1 "MountingHole_Pad" H 9550 1458 50  0001 L CNN
-F 2 "MountingHole:MountingHole_2.2mm_M2_DIN965_Pad" H 9450 1500 50  0001 C CNN
+F 2 "MountingHole:MountingHole_3.2mm_M3_DIN965_Pad" H 9450 1500 50  0001 C CNN
 F 3 "~" H 9450 1500 50  0001 C CNN
 	1    9450 1500
