File: LED_DC/LED_DC/23S17.sch (KiCad schematic (older format))
At the start: 20 parts, among them Q1 FDV304P, Q2 FDV304P, Q3 FDV304P, Q4 FDV304P, Q5 FDV304P, Q6 FDV304P, Q7 FDV304P, Q8 FDV304P, U1 74HC238, U2 ULN2803A

Commit message: Added 20 pin header for MCU LED interface in LED schematic.
Parts:
- removed DS1: RC1602A, Connector_PinHeader_2.54mm:PinHeader_1x16_P2.54mm_Vertical, symbol Display_Character:RC1602A
- added J?: MCU interface, symbol Connector_Generic:Conn_02x10_Odd_Even
Connections:
- net labels added: KEY_COL1, KEY_COL2, KEY_ROW1, KEY_ROW2
- wire segments 67 -> 74
- no-connect marks 3 -> 1
Changed lines of the file:
@@
 Text Notes 3150 7400 0    50   ~ 0
 COMM is generally used during driving Relays, for LEDs not needed
-$Comp
-L power:+5V #PWR05
-U 1 1 5FC0566D
-P 2850 1850
-F 0 "#PWR05" H 2850 1700 50  0001 C CNN
-F 1 "+5V" H 2865 2023 50  0000 C CNN
-F 2 "" H 2850 1850 50  0001 C CNN
-F 3 "" H 2850 1850 50  0001 C CNN
-	1    2850 1850
-	1    0    0    -1
-$EndComp
-Wire Wire Line
-	2850 1850 2850 1900
-$Comp
-L power:GND #PWR08
-U 1 1 5FC07527
-P 2850 3550
-F 0 "#PWR08" H 2850 3300 50  0001 C CNN
-F 1 "GND" H 2855 3377 50  0000 C CNN
-F 2 "" H 2850 3550 50  0001 C CNN
-F 3 "" H 2850 3550 50  0001 C CNN
-	1    2850 3550
-	1    0    0    -1
-$EndComp
 Wire Notes Line
 	1500 800  1500 4400
@@
 Wire Notes Line
 	5700 800  1500 800
-Wire Wire Line
-	2850 3500 2850 3550
 $Comp
 L LED_DC-rescue:DMG2305UX-13-dk_Transistors-FETs-MOSFETs-Single Q1
@@
 Wire Wire Line
 	9800 5750 9800 5650
-Text GLabel 2350 2300 0    50   Input ~ 0
-C1
-Text GLabel 2350 2400 0    50   Input ~ 0
-C2
-Text GLabel 2350 2500 0    50   Input ~ 0
-C3
-Text GLabel 2350 2600 0    50   Input ~ 0
-D0
-Text GLabel 2350 2700 0    50   Input ~ 0
-D1
-Text GLabel 2350 2800 0    50   Input ~ 0
-D2
-Text GLabel 2350 2900 0    50   Input ~ 0
-D3
-Text GLabel 2350 3000 0    50   Input ~ 0
-D4
-Text GLabel 2350 3100 0    50   Input ~ 0
-D5
-Text GLabel 2350 3200 0    50   Input ~ 0
-D6
-Text GLabel 2350 3300 0    50   Input ~ 0
-D7
-Wire Wire Line
-	2450 2600 2350 2600
-Wire Wire Line
-	2350 2700 2450 2700
-Wire Wire Line
-	2450 2800 2350 2800
-Wire Wire Line
-	2350 2900 2450 2900
-Wire Wire Line
-	2450 3000 2350 3000
-Wire Wire Line
-	2350 3100 2450 3100
-Wire Wire Line
-	2450 3200 2350 3200
-Wire Wire Line
-	2350 3300 2450 3300
 $Comp
 L power:+5V #PWR04
@@
 Wire Wire Line
 	4900 5100 4700 5100
-$Comp
-L Display_Character:RC1602A DS1
-U 1 1 5FC030D8
-P 2850 2800
-F 0 "DS1" H 3000 3650 50  0000 C CNN
-F 1 "RC1602A" H 3050 3550 50  0000 C CNN
-F 2 "Connector_PinHeader_2.54mm:PinHeader_1x16_P2.54mm_Vertical" H 2850 1900 50  0001 C CIN
-F 3 "http://www.icbank.com/data/ICBShop/board/HY1602E.pdf" H 3050 2900 50  0001 C CNN
-	1    2850 2800
-	1    0    0    -1
-$EndComp
-Text Notes 3550 2750 0    50   ~ 0
+Text Notes 2350 4100 0    50   ~ 0
 Seven Segment/LCD display Interface.
 $Comp
-L power:PWR_FLAG #FLG0101
-U 1 1 60176418
-P 2650 1900
-F 0 "#FLG0101" H 2650 1975 50  0001 C CNN
-F 1 "PWR_FLAG" V 2650 2027 50  0000 L CNN
-F 2 "" H 2650 1900 50  0001 C CNN
-F 3 "~" H 2650 1900 50  0001 C CNN
-	1    2650 1900
-	0    -1   -1   0
-$EndComp
-$Comp
-L power:PWR_FLAG #FLG0102
-U 1 1 60176CCD
-P 2600 3550
-F 0 "#FLG0102" H 2600 3625 50  0001 C CNN
-F 1 "PWR_FLAG" V 2600 3677 50  0000 L CNN
-F 2 "" H 2600 3550 50  0001 C CNN
-F 3 "~" H 2600 3550 50  0001 C CNN
-	1    2600 3550
-	0    -1   -1   0
-$EndComp
-Wire Wire Line
-	2600 3550 2850 3550
-Connection ~ 2850 3550
-Wire Wire Line
-	2650 1900 2850 1900
-Connection ~ 2850 1900
-Wire Wire Line
-	2850 1900 2850 2100
-NoConn ~ 3250 2600
-NoConn ~ 3250 3000
-NoConn ~ 3250 3100
-Wire Wire Line
-	2350 2300 2450 2300
-Wire Wire Line
-	2450 2400 2350 2400
-Wire Wire Line
-	2350 2500 2450 2500
+L Connector_Generic:Conn_02x10_Odd_Even J?
+U 1 1 6068829A
+P 2900 2950
+F 0 "J?" H 2950 3567 50  0000 C CNN
+F 1 "MCU interface" H 2950 3476 50  0000 C CNN
+F 2 "" H 2900 2950 50  0001 C CNN
+F 3 "~" H 2900 2950 50  0001 C CNN
+	1    2900 2950
+	1    0    0    -1
+$EndComp
+Text GLabel 2550 2650 0    50   Input ~ 0
+D0
+Text GLabel 3350 2650 2    50   Input ~ 0
+D1
+Text GLabel 2550 2750 0    50   Input ~ 0
+D2
+Text GLabel 3350 2750 2    50   Input ~ 0
+D3
+Text GLabel 2550 2850 0    50   Input ~ 0
+D4
+Text GLabel 3350 2850 2    50   Input ~ 0
+D5
+Text GLabel 2550 2950 0    50   Input ~ 0
+D6
+Text GLabel 3350 2950 2    50   Input ~ 0
+D7
+Text GLabel 2550 3050 0    50   Input ~ 0
+C1
+Text GLabel 3350 3050 2    50   Input ~ 0
+C2
+Text GLabel 2550 3150 0    50   Input ~ 0
+C3
+NoConn ~ 3200 3150
+Text GLabel 2550 3250 0    50   Output ~ 0
+KEY_ROW1
+Text GLabel 3350 3250 2    50   Output ~ 0
+KEY_ROW2
+Text GLabel 2550 3350 0    50   Output ~ 0
+KEY_COL1
+Text GLabel 3350 3350 2    50   Output ~ 0
+KEY_COL2
+$Comp
+L power:GND #PWR?
+U 1 1 60691F3F
+P 2550 3550
+F 0 "#PWR?" H 2550 3300 50  0001 C CNN
+F 1 "GND" H 2555 3377 50  0000 C CNN
+F 2 "" H 2550 3550 50  0001 C CNN
+F 3 "" H 2550 3550 50  0001 C CNN
+	1    2550 3550
+	1    0    0    -1
+$EndComp
+$Comp
+L power:GND #PWR?
+U 1 1 60692355
+P 3350 3550
+F 0 "#PWR?" H 3350 3300 50  0001 C CNN
+F 1 "GND" H 3355 3377 50  0000 C CNN
+F 2 "" H 3350 3550 50  0001 C CNN
+F 3 "" H 3350 3550 50  0001 C CNN
+	1    3350 3550
+	1    0    0    -1
+$EndComp
+$Comp
+L power:+5V #PWR?
+U 1 1 60692883
+P 2550 2400
+F 0 "#PWR?" H 2550 2250 50  0001 C CNN
+F 1 "+5V" H 2565 2573 50  0000 C CNN
+F 2 "" H 2550 2400 50  0001 C CNN
+F 3 "" H 2550 2400 50  0001 C CNN
+	1    2550 2400
+	1    0    0    -1
+$EndComp
+$Comp
+L power:+5V #PWR?
+U 1 1 60692BF9
+P 3350 2400
+F 0 "#PWR?" H 3350 2250 50  0001 C CNN
+F 1 "+5V" H 3365 2573 50  0000 C CNN
+F 2 "" H 3350 2400 50  0001 C CNN
+F 3 "" H 3350 2400 50  0001 C CNN
+	1    3350 2400
+	1    0    0    -1
+$EndComp
+Wire Wire Line
+	3350 2400 3350 2550
+Wire Wire Line
+	3350 2550 3200 2550
+Wire Wire Line
+	2700 2550 2550 2550
+Wire Wire Line
+	2550 2550 2550 2400
+Wire Wire Line
+	2550 2650 2700 2650
+Wire Wire Line
+	2700 2750 2550 2750
+Wire Wire Line
+	2550 2850 2700 2850
+Wire Wire Line
+	2700 2950 2550 2950
+Wire Wire Line
+	2550 3050 2700 3050
+Wire Wire Line
+	2700 3150 2550 3150
+Wire Wire Line
+	2550 3250 2700 3250
+Wire Wire Line
+	2700 3350 2550 3350
+Wire Wire Line
+	2700 3450 2550 3450
+Wire Wire Line
+	2550 3450 2550 3550
+Wire Wire Line
+	3200 3450 3350 3450
+Wire Wire Line
+	3350 3450 3350 3550
+Wire Wire Line
+	3350 3350 3200 3350
+Wire Wire Line
+	3200 3250 3350 3250
+Wire Wire Line
+	3350 3050 3200 3050
+Wire Wire Line
+	3200 2950 3350 2950
+Wire Wire Line
+	3350 2850 3200 2850
+Wire Wire Line
+	3200 2750 3350 2750
+Wire Wire Line
+	3350 2650 3200 2650
 $EndSCHEMATC

Commit message: Updated PCB.
Parts:
- J1: renamed from J?; footprint (none) -> Connector_PinHeader_2.54mm:PinHeader_2x10_P2.54mm_Vertical
Changed lines of the file:
@@
 Seven Segment/LCD display Interface.
 $Comp
-L Connector_Generic:Conn_02x10_Odd_Even J?
+L Connector_Generic:Conn_02x10_Odd_Even J1
 U 1 1 6068829A
 P 2900 2950
-F 0 "J?" H 2950 3567 50  0000 C CNN
+F 0 "J1" H 2950 3567 50  0000 C CNN
 F 1 "MCU interface" H 2950 3476 50  0000 C CNN
-F 2 "" H 2900 2950 50  0001 C CNN
+F 2 "Connector_PinHeader_2.54mm:PinHeader_2x10_P2.54mm_Vertical" H 2900 2950 50  0001 C CNN
 F 3 "~" H 2900 2950 50  0001 C CNN
 	1    2900 2950
@@
 KEY_COL2
 $Comp
-L power:GND #PWR?
+L power:GND #PWR02
 U 1 1 60691F3F
 P 2550 3550
-F 0 "#PWR?" H 2550 3300 50  0001 C CNN
+F 0 "#PWR02" H 2550 3300 50  0001 C CNN
 F 1 "GND" H 2555 3377 50  0000 C CNN
 F 2 "" H 2550 3550 50  0001 C CNN
@@
 $EndComp
 $Comp
-L power:GND #PWR?
+L power:GND #PWR05
 U 1 1 60692355
 P 3350 3550
-F 0 "#PWR?" H 3350 3300 50  0001 C CNN
+F 0 "#PWR05" H 3350 3300 50  0001 C CNN
 F 1 "GND" H 3355 3377 50  0000 C CNN
 F 2 "" H 3350 3550 50  0001 C CNN
@@
 $EndComp
 $Comp
-L power:+5V #PWR?
+L power:+5V #PWR01
 U 1 1 60692883
 P 2550 2400
-F 0 "#PWR?" H 2550 2250 50  0001 C CNN
+F 0 "#PWR01" H 2550 2250 50  0001 C CNN
 F 1 "+5V" H 2565 2573 50  0000 C CNN
 F 2 "" H 2550 2400 50  0001 C CNN
@@
 $EndComp
 $Comp
-L power:+5V #PWR?
+L power:+5V #PWR03
 U 1 1 60692BF9
 P 3350 2400
-F 0 "#PWR?" H 3350 2250 50  0001 C CNN
+F 0 "#PWR03" H 3350 2250 50  0001 C CNN
 F 1 "+5V" H 3365 2573 50  0000 C CNN
 F 2 "" H 3350 2400 50  0001 C CNN
@@
 Wire Wire Line
 	3350 2650 3200 2650
+$Comp
+L power:PWR_FLAG #FLG0101
+U 1 1 606A139D
+P 3550 2550
+F 0 "#FLG0101" H 3550 2625 50  0001 C CNN
+F 1 "PWR_FLAG" V 3550 2678 50  0000 L CNN
+F 2 "" H 3550 2550 50  0001 C CNN
+F 3 "~" H 3550 2550 50  0001 C CNN
+	1    3550 2550
+	0    1    1    0
+$EndComp
+$Comp
+L power:PWR_FLAG #FLG0102
+U 1 1 606A16E2
+P 3550 3450
+F 0 "#FLG0102" H 3550 3525 50  0001 C CNN
+F 1 "PWR_FLAG" V 3550 3578 50  0000 L CNN
+F 2 "" H 3550 3450 50  0001 C CNN
+F 3 "~" H 3550 3450 50  0001 C CNN
+	1    3550 3450
+	0    1    1    0
+$EndComp
+Wire Wire Line
+	3550 3450 3350 3450
+Connection ~ 3350 3450
+Wire Wire Line
+	3350 2550 3550 2550
+Connection ~ 3350 2550
 $EndSCHEMATC

Commit message: Updated the LED DC PCB.
Parts:
- removed Q4, Q7: FDV304P, Package_TO_SOT_SMD:SOT-23_Handsoldering, symbol LED_DC-rescue:DMG2305UX-13-dk_Transistors-FETs-MOSFETs-Single
- Q1, Q2, Q3, Q5, Q6, Q8: symbol LED_DC-rescue:DMG2305UX-13-dk_Transistors-FETs-MOSFETs-Single -> LED_DC-rescue:DMG2305UX-13-dk_Transistors-FETs-MOSFETs-Single-LED_DC-rescue
Changed lines of the file:
@@
 	5700 800  1500 800
 $Comp
-L LED_DC-rescue:DMG2305UX-13-dk_Transistors-FETs-MOSFETs-Single Q1
+L LED_DC-rescue:DMG2305UX-13-dk_Transistors-FETs-MOSFETs-Single-LED_DC-rescue Q1
 U 1 1 5FAF9A47
 P 8100 1250
@@
 D_C_2
 $Comp
-L LED_DC-rescue:DMG2305UX-13-dk_Transistors-FETs-MOSFETs-Single Q?
+L LED_DC-rescue:DMG2305UX-13-dk_Transistors-FETs-MOSFETs-Single-LED_DC-rescue Q?
 U 1 1 5FDA9743
 P 9800 1250
@@
 D_C_3
 $Comp
-L LED_DC-rescue:DMG2305UX-13-dk_Transistors-FETs-MOSFETs-Single Q?
+L LED_DC-rescue:DMG2305UX-13-dk_Transistors-FETs-MOSFETs-Single-LED_DC-rescue Q?
 U 1 1 5FDAF306
 P 8100 2400
@@
 D_C_4
 $Comp
-L LED_DC-rescue:DMG2305UX-13-dk_Transistors-FETs-MOSFETs-Single Q?
+L LED_DC-rescue:DMG2305UX-13-dk_Transistors-FETs-MOSFETs-Single-LED_DC-rescue Q?
 U 1 1 5FDAF320
 P 9800 2400
@@
 Wire Wire Line
 	9800 2700 9800 2600
-Text GLabel 8500 4200 2    50   Input ~ 0
-D_C_5
-$Comp
-L LED_DC-rescue:DMG2305UX-13-dk_Transistors-FETs-MOSFETs-Single Q?
-U 1 1 5FDB7FD3
-P 8100 4300
-AR Path="/5FDB7FD3" Ref="Q?"  Part="1"
-AR Path="/5FC37B24/5FDB7FD3" Ref="Q3"  Part="1"
-F 0 "Q3" H 8208 4353 60  0000 L CNN
-F 1 "FDV304P" H 8208 4247 60  0000 L CNN
-F 2 "Package_TO_SOT_SMD:SOT-23_Handsoldering" H 8300 4500 60  0001 L CNN
-F 3 "https://www.diodes.com/assets/Datasheets/DMG2305UX.pdf" H 8300 4600 60  0001 L CNN
-F 4 "DMG2305UX-13DICT-ND" H 8300 4700 60  0001 L CNN "Digi-Key_PN"
-F 5 "DMG2305UX-13" H 8300 4800 60  0001 L CNN "MPN"
-F 6 "Discrete Semiconductor Products" H 8300 4900 60  0001 L CNN "Category"
-F 7 "Transistors - FETs, MOSFETs - Single" H 8300 5000 60  0001 L CNN "Family"
-F 8 "https://www.diodes.com/assets/Datasheets/DMG2305UX.pdf" H 8300 5100 60  0001 L CNN "DK_Datasheet_Link"
-F 9 "/product-detail/en/diodes-incorporated/DMG2305UX-13/DMG2305UX-13DICT-ND/4251589" H 8300 5200 60  0001 L CNN "DK_Detail_Page"
-F 10 "MOSFET P-CH 20V 4.2A SOT23" H 8300 5300 60  0001 L CNN "Description"
-F 11 "Diodes Incorporated" H 8300 5400 60  0001 L CNN "Manufacturer"
-F 12 "Active" H 8300 5500 60  0001 L CNN "Status"
-	1    8100 4300
-	-1   0    0    1
-$EndComp
-$Comp
-L power:+5V #PWR017
-U 1 1 5FDB7FD9
-P 8100 4000
-F 0 "#PWR017" H 8100 3850 50  0001 C CNN
-F 1 "+5V" H 8115 4173 50  0000 C CNN
-F 2 "" H 8100 4000 50  0001 C CNN
-F 3 "" H 8100 4000 50  0001 C CNN
-	1    8100 4000
-	1    0    0    -1
-$EndComp
-Wire Wire Line
-	8100 4000 8100 4100
-Wire Wire Line
-	8400 4200 8500 4200
-Text GLabel 8100 4600 3    50   Output ~ 0
-D_5
-Wire Wire Line
-	8100 4600 8100 4500
-Text GLabel 10200 4200 2    50   Input ~ 0
-D_C_6
-$Comp
-L LED_DC-rescue:DMG2305UX-13-dk_Transistors-FETs-MOSFETs-Single Q?
-U 1 1 5FDB7FED
-P 9800 4300
-AR Path="/5FDB7FED" Ref="Q?"  Part="1"
-AR Path="/5FC37B24/5FDB7FED" Ref="Q7"  Part="1"
-F 0 "Q7" H 9908 4353 60  0000 L CNN
-F 1 "FDV304P" H 9908 4247 60  0000 L CNN
-F 2 "Package_TO_SOT_SMD:SOT-23_Handsoldering" H 10000 4500 60  0001 L CNN
-F 3 "https://www.diodes.com/assets/Datasheets/DMG2305UX.pdf" H 10000 4600 60  0001 L CNN
-F 4 "DMG2305UX-13DICT-ND" H 10000 4700 60  0001 L CNN "Digi-Key_PN"
-F 5 "DMG2305UX-13" H 10000 4800 60  0001 L CNN "MPN"
-F 6 "Discrete Semiconductor Products" H 10000 4900 60  0001 L CNN "Category"
-F 7 "Transistors - FETs, MOSFETs - Single" H 10000 5000 60  0001 L CNN "Family"
-F 8 "https://www.diodes.com/assets/Datasheets/DMG2305UX.pdf" H 10000 5100 60  0001 L CNN "DK_Datasheet_Link"
-F 9 "/product-detail/en/diodes-incorporated/DMG2305UX-13/DMG2305UX-13DICT-ND/4251589" H 10000 5200 60  0001 L CNN "DK_Detail_Page"
-F 10 "MOSFET P-CH 20V 4.2A SOT23" H 10000 5300 60  0001 L CNN "Description"
-F 11 "Diodes Incorporated" H 10000 5400 60  0001 L CNN "Manufacturer"
-F 12 "Active" H 10000 5500 60  0001 L CNN "Status"
-	1    9800 4300
-	-1   0    0    1
-$EndComp
-$Comp
-L power:+5V #PWR021
-U 1 1 5FDB7FF3
-P 9800 4000
-F 0 "#PWR021" H 9800 3850 50  0001 C CNN
-F 1 "+5V" H 9815 4173 50  0000 C CNN
-F 2 "" H 9800 4000 50  0001 C CNN
-F 3 "" H 9800 4000 50  0001 C CNN
-	1    9800 4000
-	1    0    0    -1
-$EndComp
-Wire Wire Line
-	9800 4000 9800 4100
-Wire Wire Line
-	10100 4200 10200 4200
-Text GLabel 9800 4600 3    50   Output ~ 0
-D_6
-Wire Wire Line
-	9800 4600 9800 4500
-Text GLabel 8500 5350 2    50   Input ~ 0
-D_C_7
-$Comp
-L LED_DC-rescue:DMG2305UX-13-dk_Transistors-FETs-MOSFETs-Single Q?
-U 1 1 5FDB8007
-P 8100 5450
-AR Path="/5FDB8007" Ref="Q?"  Part="1"
-AR Path="/5FC37B24/5FDB8007" Ref="Q4"  Part="1"
-F 0 "Q4" H 8208 5503 60  0000 L CNN
-F 1 "FDV304P" H 8208 5397 60  0000 L CNN
-F 2 "Package_TO_SOT_SMD:SOT-23_Handsoldering" H 8300 5650 60  0001 L CNN
-F 3 "https://www.diodes.com/assets/Datasheets/DMG2305UX.pdf" H 8300 5750 60  0001 L CNN
-F 4 "DMG2305UX-13DICT-ND" H 8300 5850 60  0001 L CNN "Digi-Key_PN"
-F 5 "DMG2305UX-13" H 8300 5950 60  0001 L CNN "MPN"
-F 6 "Discrete Semiconductor Products" H 8300 6050 60  0001 L CNN "Category"
-F 7 "Transistors - FETs, MOSFETs - Single" H 8300 6150 60  0001 L CNN "Family"
-F 8 "https://www.diodes.com/assets/Datasheets/DMG2305UX.pdf" H 8300 6250 60  0001 L CNN "DK_Datasheet_Link"
-F 9 "/product-detail/en/diodes-incorporated/DMG2305UX-13/DMG2305UX-13DICT-ND/4251589" H 8300 6350 60  0001 L CNN "DK_Detail_Page"
-F 10 "MOSFET P-CH 20V 4.2A SOT23" H 8300 6450 60  0001 L CNN "Description"
-F 11 "Diodes Incorporated" H 8300 6550 60  0001 L CNN "Manufacturer"
-F 12 "Active" H 8300 6650 60  0001 L CNN "Status"
-	1    8100 5450
-	-1   0    0    1
-$EndComp
-$Comp
-L power:+5V #PWR018
-U 1 1 5FDB800D
-P 8100 5150
-F 0 "#PWR018" H 8100 5000 50  0001 C CNN
-F 1 "+5V" H 8115 5323 50  0000 C CNN
-F 2 "" H 8100 5150 50  0001 C CNN
-F 3 "" H 8100 5150 50  0001 C CNN
-	1    8100 5150
-	1    0    0    -1
-$EndComp
-Wire Wire Line
-	8100 5150 8100 5250
-Wire Wire Line
-	8400 5350 8500 5350
-Text GLabel 8100 5750 3    50   Output ~ 0
-D_7
-Wire Wire Line
-	8100 5750 8100 5650
 Text GLabel 10200 5350 2    50   Input ~ 0
 D_C_8
 $Comp
-L LED_DC-rescue:DMG2305UX-13-dk_Transistors-FETs-MOSFETs-Single Q?
+L LED_DC-rescue:DMG2305UX-13-dk_Transistors-FETs-MOSFETs-Single-LED_DC-rescue Q?
 U 1 1 5FDB8021
 P 9800 5450
@@
 	3350 2550 3550 2550
 Connection ~ 3350 2550
+Wire Wire Line
+	8100 4600 8100 4500
+Text GLabel 8100 4600 3    50   Output ~ 0
+D_5
+Wire Wire Line
+	8400 4200 8500 4200
+Wire Wire Line
+	8100 4000 8100 4100
+$Comp
+L power:+5V #PWR017
+U 1 1 5FDB7FD9
+P 8100 4000
+F 0 "#PWR017" H 8100 3850 50  0001 C CNN
+F 1 "+5V" H 8115 4173 50  0000 C CNN
+F 2 "" H 8100 4000 50  0001 C CNN
+F 3 "" H 8100 4000 50  0001 C CNN
+	1    8100 4000
+	1    0    0    -1
+$EndComp
+$Comp
+L LED_DC-rescue:DMG2305UX-13-dk_Transistors-FETs-MOSFETs-Single-LED_DC-rescue Q?
+U 1 1 5FDB7FD3
+P 8100 4300
+AR Path="/5FDB7FD3" Ref="Q?"  Part="1"
+AR Path="/5FC37B24/5FDB7FD3" Ref="Q3"  Part="1"
+F 0 "Q3" H 8208 4353 60  0000 L CNN
+F 1 "FDV304P" H 8208 4247 60  0000 L CNN
+F 2 "Package_TO_SOT_SMD:SOT-23_Handsoldering" H 8300 4500 60  0001 L CNN
+F 3 "https://www.diodes.com/assets/Datasheets/DMG2305UX.pdf" H 8300 4600 60  0001 L CNN
+F 4 "DMG2305UX-13DICT-ND" H 8300 4700 60  0001 L CNN "Digi-Key_PN"
+F 5 "DMG2305UX-13" H 8300 4800 60  0001 L CNN "MPN"
+F 6 "Discrete Semiconductor Products" H 8300 4900 60  0001 L CNN "Category"
+F 7 "Transistors - FETs, MOSFETs - Single" H 8300 5000 60  0001 L CNN "Family"
+F 8 "https://www.diodes.com/assets/Datasheets/DMG2305UX.pdf" H 8300 5100 60  0001 L CNN "DK_Datasheet_Link"
+F 9 "/product-detail/en/diodes-incorporated/DMG2305UX-13/DMG2305UX-13DICT-ND/4251589" H 8300 5200 60  0001 L CNN "DK_Detail_Page"
+F 10 "MOSFET P-CH 20V 4.2A SOT23" H 8300 5300 60  0001 L CNN "Description"
+F 11 "Diodes Incorporated" H 8300 5400 60  0001 L CNN "Manufacturer"
+F 12 "Active" H 8300 5500 60  0001 L CNN "Status"
+	1    8100 4300
+	-1   0    0    1
+$EndComp
+Text GLabel 8500 4200 2    50   Input ~ 0
+D_C_5
 $EndSCHEMATC
