File: LED_DC/LED_DC/SevenSegment.sch (KiCad schematic (older format))
At the start: 13 parts, among them U3 KCSA02-136, U4 KCSA02-136, U5 KCSA02-136, U6 KCSA02-136, U7 KCSA02-136

Commit message: Updated component values.
Parts:
- D1, D2, D3, D4, D5, D6, D7, D8: value LED -> RED-LED-3MM
Changed lines of the file:
@@
 P 4750 4800
 F 0 "D2" H 4743 5017 50  0000 C CNN
-F 1 "LED" H 4743 4926 50  0000 C CNN
+F 1 "RED-LED-3MM" H 4743 4926 50  0000 C CNN
 F 2 "LED_THT:LED_D3.0mm" H 4750 4800 50  0001 C CNN
 F 3 "~" H 4750 4800 50  0001 C CNN
@@
 P 5850 4350
 F 0 "D5" H 5843 4567 50  0000 C CNN
-F 1 "LED" H 5843 4476 50  0000 C CNN
+F 1 "RED-LED-3MM" H 5843 4476 50  0000 C CNN
 F 2 "LED_THT:LED_D3.0mm" H 5850 4350 50  0001 C CNN
 F 3 "~" H 5850 4350 50  0001 C CNN
@@
 P 4750 4450
 F 0 "D1" H 4743 4667 50  0000 C CNN
-F 1 "LED" H 4743 4576 50  0000 C CNN
+F 1 "RED-LED-3MM" H 4743 4576 50  0000 C CNN
 F 2 "LED_THT:LED_D3.0mm" H 4750 4450 50  0001 C CNN
 F 3 "~" H 4750 4450 50  0001 C CNN
@@
 P 4750 5150
 F 0 "D3" H 4743 5367 50  0000 C CNN
-F 1 "LED" H 4743 5276 50  0000 C CNN
+F 1 "RED-LED-3MM" H 4743 5276 50  0000 C CNN
 F 2 "LED_THT:LED_D3.0mm" H 4750 5150 50  0001 C CNN
 F 3 "~" H 4750 5150 50  0001 C CNN
@@
 P 4750 5500
 F 0 "D4" H 4743 5717 50  0000 C CNN
-F 1 "LED" H 4743 5626 50  0000 C CNN
+F 1 "RED-LED-3MM" H 4743 5626 50  0000 C CNN
 F 2 "LED_THT:LED_D3.0mm" H 4750 5500 50  0001 C CNN
 F 3 "~" H 4750 5500 50  0001 C CNN
@@
 P 5850 4750
 F 0 "D6" H 5843 4967 50  0000 C CNN
-F 1 "LED" H 5843 4876 50  0000 C CNN
+F 1 "RED-LED-3MM" H 5843 4876 50  0000 C CNN
 F 2 "LED_THT:LED_D3.0mm" H 5850 4750 50  0001 C CNN
 F 3 "~" H 5850 4750 50  0001 C CNN
@@
 P 5850 5100
 F 0 "D7" H 5843 5317 50  0000 C CNN
-F 1 "LED" H 5843 5226 50  0000 C CNN
+F 1 "RED-LED-3MM" H 5843 5226 50  0000 C CNN
 F 2 "LED_THT:LED_D3.0mm" H 5850 5100 50  0001 C CNN
 F 3 "~" H 5850 5100 50  0001 C CNN
@@
 P 5850 5500
 F 0 "D8" H 5843 5717 50  0000 C CNN
-F 1 "LED" H 5843 5626 50  0000 C CNN
+F 1 "RED-LED-3MM" H 5843 5626 50  0000 C CNN
 F 2 "LED_THT:LED_D3.0mm" H 5850 5500 50  0001 C CNN
 F 3 "~" H 5850 5500 50  0001 C CNN
